Commit message: Added fill body and wheel tree barebones

File: curiosity_mars_rover_description/urdf/chassis.xacro (robot description, xacro)
@@ -13,12 +13,12 @@
 					rpy="0 0 0"/>
 			<geometry>
-				<mesh filename="package://curiosity_mars_rover_description/meshes/MSL_dirty_mod_chassis_fixed.dae" scale="${scale_XYZ} ${scale_XYZ} ${scale_XYZ}"/>
-			</geometry>
-		</collision>
-		<visual>
-			<origin xyz="0 0 0"
-					rpy="0 0 0"/>
-			<geometry>
-				<mesh filename="package://curiosity_mars_rover_description/meshes/MSL_dirty_mod_chassis_fixed.dae" scale="${scale_XYZ} ${scale_XYZ} ${scale_XYZ}"/>
+				<mesh filename="package://curiosity_mars_rover_description/meshes/chassis_full_fixed_glitch_v2.dae" scale="${scale_XYZ} ${scale_XYZ} ${scale_XYZ}"/>
+			</geometry>
+		</collision>
+		<visual>
+			<origin xyz="0 0 0"
+					rpy="0 0 0"/>
+			<geometry>
+				<mesh filename="package://curiosity_mars_rover_description/meshes/chassis_full_fixed_glitch_v2.dae" scale="${scale_XYZ} ${scale_XYZ} ${scale_XYZ}"/>
 			</geometry>
 		</visual>
@@ -29,9 +29,317 @@
 			<box_inertia
 				m="${chassisMass}"
-				x="${chassisLength*scale_XYZ}"
-				y="${chassisWidth*scale_XYZ}"
+				x="${chassisWidth*scale_XYZ}"
+				y="${chassisLength*scale_XYZ}"
 				z="${chassisHeight*scale_XYZ}"/>
 		</inertial>
 	</link>
+  	<link name='left_axis'>
+		<collision>
+			<origin xyz="0 0 0"
+					rpy="0 0 0"/>
+			<geometry>
+				<mesh filename="package://curiosity_mars_rover_description/meshes/left_axis_jointfix_v2.dae" scale="${scale_XYZ} ${scale_XYZ} ${scale_XYZ}"/>
+			</geometry>
+		</collision>
+		<visual>
+			<origin xyz="0 0 0"
+					rpy="0 0 0"/>
+			<geometry>
+				<mesh filename="package://curiosity_mars_rover_description/meshes/left_axis_jointfix_v2.dae" scale="${scale_XYZ} ${scale_XYZ} ${scale_XYZ}"/>
+			</geometry>
+		</visual>
+		<inertial>
+			<origin xyz="0 0 0"
+					rpy="0 0 0"/>
+			<mass value="${axisMass}"/>
+			<box_inertia
+				m="${axisMass}"
+				x="${axisWidth*scale_XYZ}"
+				y="${axisLength*scale_XYZ}"
+				z="${axisHeight*scale_XYZ}"/>
+		</inertial>
+	</link>
+  	<joint name="left_axis_joint" type="fixed">
+		<parent link="chassis"/>
+		<child link="left_axis"/>
+		<origin xyz="0.7938 -0.2133 0" rpy="0 -0.19565141 0"/>
+	</joint>
+  	<link name='suspension_arm_F_L'>
+		<collision>
+			<origin xyz="0 0 0"
+					rpy="0 0 0"/>
+			<geometry>
+				<mesh filename="package://curiosity_mars_rover_description/meshes/suspension_arm_F_L_fixed.dae" scale="${scale_XYZ} ${scale_XYZ} ${scale_XYZ}"/>
+			</geometry>
+		</collision>
+		<visual>
+			<origin xyz="0 0 0"
+					rpy="0 0 0"/>
+			<geometry>
+				<mesh filename="package://curiosity_mars_rover_description/meshes/suspension_arm_F_L_fixed.dae" scale="${scale_XYZ} ${scale_XYZ} ${scale_XYZ}"/>
+			</geometry>
+		</visual>
+		<inertial>
+			<origin xyz="0 0 0"
+					rpy="0 0 0"/>
+			<mass value="${suspension_arm_F_Mass}"/>
+			<box_inertia
+				m="${suspension_arm_F_Mass}"
+				x="${suspension_arm_F_Width*scale_XYZ}"
+				y="${suspension_arm_F_Length*scale_XYZ}"
+				z="${suspension_arm_F_Height*scale_XYZ}"/>
+		</inertial>
+	</link>
+  	<joint name="suspension_arm_F_L_joint" type="revolute">
+		<parent link="left_axis"/>
+		<child link="suspension_arm_F_L"/>
+		<origin xyz="0 0 0" rpy="0 0 0"/>
+		<limit lower="-0.2" upper="0.2" effort="10000.0" velocity="100.0"/>
+        <axis xyz="1 0 0"/>
+	</joint>
+	<link name='suspension_arm_B_L'>
+		<collision>
+			<origin xyz="0 0 0"
+					rpy="0 0 0"/>
+			<geometry>
+				<mesh filename="package://curiosity_mars_rover_description/meshes/suspension_arm_B_L_fixed.dae" scale="${scale_XYZ} ${scale_XYZ} ${scale_XYZ}"/>
+			</geometry>
+		</collision>
+		<visual>
+			<origin xyz="0 0 0"
+					rpy="0 0 0"/>
+			<geometry>
+				<mesh filename="package://curiosity_mars_rover_description/meshes/suspension_arm_B_L_fixed.dae" scale="${scale_XYZ} ${scale_XYZ} ${scale_XYZ}"/>
+			</geometry>
+		</visual>
+		<inertial>
+			<origin xyz="0 0 0"
+					rpy="0 0 0"/>
+			<mass value="${suspension_arm_F_Mass}"/>
+			<box_inertia
+				m="${suspension_arm_F_Mass}"
+				x="${suspension_arm_F_Width*scale_XYZ}"
+				y="${suspension_arm_F_Length*scale_XYZ}"
+				z="${suspension_arm_F_Height*scale_XYZ}"/>
+		</inertial>
+	</link>
+  	<joint name="suspension_arm_B_L_joint" type="revolute">
+		<parent link="left_axis"/>
+		<child link="suspension_arm_B_L"/>
+		<origin xyz="0 0 0" rpy="0 0 0"/>
+		<limit lower="-0.2" upper="0.2" effort="10000.0" velocity="100.0"/>
+        <axis xyz="1 0 0"/>
+	</joint>
+ 	<link name='suspension_arm_B_L_to_B2_L'>
+		<inertial>
+            <origin xyz="0 0 0" rpy="0 0 0"/>
+            <mass value="0.02" />
+            <inertia ixx="2.61666666667e-05" ixy="0.0" ixz="0.0" iyy="2.61666666667e-05" iyz="0.0" izz="3.6e-05"/>
+        </inertial>
+        <collision>
+            <origin xyz="0 0 0.015" rpy="0 0 0"/>
+            <geometry>
+                <cylinder radius="0.06" length="0.035"/>
+            </geometry>
+        </collision>
+		<visual>
+            <origin rpy="0.0 1.57 0" xyz="0 0 0"/>
+            <geometry>
+                <cylinder radius="0.04" length="0.1"/>
+            </geometry>
+        </visual>
+	</link>
+	<joint name="suspension_arm_B_L_to_B2_L_joint" type="fixed">
+		<parent link="suspension_arm_B_L"/>
+		<child link="suspension_arm_B_L_to_B2_L"/>
+		<origin xyz="-0.05159 0.73683 -0.22972" rpy="0 0.1937315 0"/>
+	</joint>
+	<link name='suspension_arm_B2_L'>
+		<collision>
+			<origin xyz="0 0 0"
+					rpy="0 0 0"/>
+			<geometry>
+				<mesh filename="package://curiosity_mars_rover_description/meshes/suspension_arm_B2_L_fixed.dae" scale="${scale_XYZ} ${scale_XYZ} ${scale_XYZ}"/>
+			</geometry>
+		</collision>
+		<visual>
+			<origin xyz="0 0 0"
+					rpy="0 0 0"/>
+			<geometry>
+				<mesh filename="package://curiosity_mars_rover_description/meshes/suspension_arm_B2_L_fixed.dae" scale="${scale_XYZ} ${scale_XYZ} ${scale_XYZ}"/>
+			</geometry>
+		</visual>
+		<inertial>
+			<origin xyz="0 0 0"
+					rpy="0 0 0"/>
+			<mass value="${suspension_arm_F_Mass}"/>
+			<box_inertia
+				m="${suspension_arm_F_Mass}"
+				x="${suspension_arm_F_Width*scale_XYZ}"
+				y="${suspension_arm_F_Length*scale_XYZ}"
+				z="${suspension_arm_F_Height*scale_XYZ}"/>
+		</inertial>
+	</link>
+  	<joint name="suspension_arm_B2_L_joint" type="revolute">
+		<parent link="suspension_arm_B_L_to_B2_L"/>
+		<child link="suspension_arm_B2_L"/>
+		<origin xyz="0 0 0" rpy="0 0 0"/>
+		<limit lower="-0.2" upper="0.2" effort="10000.0" velocity="100.0"/>
+        <axis xyz="1 0 0"/>
+	</joint>
+  	<link name='right_axis'>
+		<collision>
+			<origin xyz="0 0 0"
+					rpy="0 0 0"/>
+			<geometry>
+				<mesh filename="package://curiosity_mars_rover_description/meshes/right_axis_jointfix_v2.dae" scale="${scale_XYZ} ${scale_XYZ} ${scale_XYZ}"/>
+			</geometry>
+		</collision>
+		<visual>
+			<origin xyz="0 0 0"
+					rpy="0 0 0"/>
+			<geometry>
+				<mesh filename="package://curiosity_mars_rover_description/meshes/right_axis_jointfix_v2.dae" scale="${scale_XYZ} ${scale_XYZ} ${scale_XYZ}"/>
+			</geometry>
+		</visual>
+		<inertial>
+			<origin xyz="0 0 0"
+					rpy="0 0 0"/>
+			<mass value="${axisMass}"/>
+			<box_inertia
+				m="${axisMass}"
+				x="${axisWidth*scale_XYZ}"
+				y="${axisLength*scale_XYZ}"
+				z="${axisHeight*scale_XYZ}"/>
+		</inertial>
+	</link>
+  	<joint name="right_axis_joint" type="fixed">
+		<parent link="chassis"/>
+		<child link="right_axis"/>
+		<origin xyz="-0.7938 -0.2133 0" rpy="0 0.19565141 0"/>
+	</joint>
+	<link name='suspension_arm_F_R'>
+		<collision>
+			<origin xyz="0 0 0"
+					rpy="0 0 0"/>
+			<geometry>
+				<mesh filename="package://curiosity_mars_rover_description/meshes/suspension_arm_F_R_fixed.dae" scale="${scale_XYZ} ${scale_XYZ} ${scale_XYZ}"/>
+			</geometry>
+		</collision>
+		<visual>
+			<origin xyz="0 0 0"
+					rpy="0 0 0"/>
+			<geometry>
+				<mesh filename="package://curiosity_mars_rover_description/meshes/suspension_arm_F_R_fixed.dae" scale="${scale_XYZ} ${scale_XYZ} ${scale_XYZ}"/>
+			</geometry>
+		</visual>
+		<inertial>
+			<origin xyz="0 0 0"
+					rpy="0 0 0"/>
+			<mass value="${suspension_arm_F_Mass}"/>
+			<box_inertia
+				m="${suspension_arm_F_Mass}"
+				x="${suspension_arm_F_Width*scale_XYZ}"
+				y="${suspension_arm_F_Length*scale_XYZ}"
+				z="${suspension_arm_F_Height*scale_XYZ}"/>
+		</inertial>
+	</link>
+  	<joint name="suspension_arm_F_R_joint" type="revolute">
+		<parent link="right_axis"/>
+		<child link="suspension_arm_F_R"/>
+		<origin xyz="0 0 0" rpy="0 0 0"/>
+		<limit lower="-0.2" upper="0.2" effort="10000.0" velocity="100.0"/>
+        <axis xyz="1 0 0"/>
+	</joint>
+	<link name='suspension_arm_B_R'>
+		<collision>
+			<origin xyz="0 0 0"
+					rpy="0 0 0"/>
+			<geometry>
+				<mesh filename="package://curiosity_mars_rover_description/meshes/suspension_arm_B_R_fixed.dae" scale="${scale_XYZ} ${scale_XYZ} ${scale_XYZ}"/>
+			</geometry>
+		</collision>
+		<visual>
+			<origin xyz="0 0 0"
+					rpy="0 0 0"/>
+			<geometry>
+				<mesh filename="package://curiosity_mars_rover_description/meshes/suspension_arm_B_R_fixed.dae" scale="${scale_XYZ} ${scale_XYZ} ${scale_XYZ}"/>
+			</geometry>
+		</visual>
+		<inertial>
+			<origin xyz="0 0 0"
+					rpy="0 0 0"/>
+			<mass value="${suspension_arm_F_Mass}"/>
+			<box_inertia
+				m="${suspension_arm_F_Mass}"
+				x="${suspension_arm_F_Width*scale_XYZ}"
+				y="${suspension_arm_F_Length*scale_XYZ}"
+				z="${suspension_arm_F_Height*scale_XYZ}"/>
+		</inertial>
+	</link>
+  	<joint name="suspension_arm_B_R_joint" type="revolute">
+		<parent link="right_axis"/>
+		<child link="suspension_arm_B_R"/>
+		<origin xyz="0 0 0" rpy="0 0 0"/>
+		<limit lower="-0.2" upper="0.2" effort="10000.0" velocity="100.0"/>
+        <axis xyz="1 0 0"/>
+	</joint>
+  	<link name='suspension_arm_B_R_to_B2_R'>
+		<inertial>
+            <origin xyz="0 0 0" rpy="0 0 0"/>
+            <mass value="0.02" />
+            <inertia ixx="2.61666666667e-05" ixy="0.0" ixz="0.0" iyy="2.61666666667e-05" iyz="0.0" izz="3.6e-05"/>
+        </inertial>
+        <collision>
+            <origin xyz="0 0 0.015" rpy="0 0 0"/>
+            <geometry>
+                <cylinder radius="0.06" length="0.035"/>
+            </geometry>
+        </collision>
+		<visual>
+            <origin rpy="0.0 1.57 0" xyz="0 0 0"/>
+            <geometry>
+                <cylinder radius="0.04" length="0.1"/>
+            </geometry>
+        </visual>
+	</link>
+	<joint name="suspension_arm_B_R_to_B2_R_joint" type="fixed">
+		<parent link="suspension_arm_B_R"/>
+		<child link="suspension_arm_B_R_to_B2_R"/>
+		<origin xyz="0.05159 0.73683 -0.22972" rpy="0 -0.1937315 0"/>
+	</joint>
+	<link name='suspension_arm_B2_R'>
+		<collision>
+			<origin xyz="0 0 0"
+					rpy="0 0 0"/>
+			<geometry>
+				<mesh filename="package://curiosity_mars_rover_description/meshes/suspension_arm_B2_R_fixed.dae" scale="${scale_XYZ} ${scale_XYZ} ${scale_XYZ}"/>
+			</geometry>
+		</collision>
+		<visual>
+			<origin xyz="0 0 0"
+					rpy="0 0 0"/>
+			<geometry>
+				<mesh filename="package://curiosity_mars_rover_description/meshes/suspension_arm_B2_R_fixed.dae" scale="${scale_XYZ} ${scale_XYZ} ${scale_XYZ}"/>
+			</geometry>
+		</visual>
+		<inertial>
+			<origin xyz="0 0 0"
+					rpy="0 0 0"/>
+			<mass value="${suspension_arm_F_Mass}"/>
+			<box_inertia
+				m="${suspension_arm_F_Mass}"
+				x="${suspension_arm_F_Width*scale_XYZ}"
+				y="${suspension_arm_F_Length*scale_XYZ}"
+				z="${suspension_arm_F_Height*scale_XYZ}"/>
+		</inertial>
+	</link>
+  	<joint name="suspension_arm_B2_R_joint" type="revolute">
+		<parent link="suspension_arm_B_R_to_B2_R"/>
+		<child link="suspension_arm_B2_R"/>
+		<origin xyz="0 0 0" rpy="0 0 0"/>
+		<limit lower="-0.2" upper="0.2" effort="10000.0" velocity="100.0"/>
+        <axis xyz="1 0 0"/>
+	</joint>
   </xacro:macro>
 </robot>

File: curiosity_mars_rover_description/urdf/curiosity_mars_rover_properties.xacro (robot description, xacro)
@@ -6,8 +6,21 @@
 	<xacro:property name="scale_XYZ" value="1.0"/>
 	<!-- Chassis properties -->
+	<!--
+	<xacro:property name="chassisHeight" value="0.76"/>
+	<xacro:property name="chassisLength" value="1.53774"/>
+	<xacro:property name="chassisWidth" value="2.08157"/>
+	-->
 	<xacro:property name="chassisHeight" value="0.76"/>
 	<xacro:property name="chassisLength" value="2.08157"/>
 	<xacro:property name="chassisWidth" value="1.53774"/>
 	<xacro:property name="chassisMass" value="20.0"/>
+	<xacro:property name="axisHeight" value="0.36388"/>
+	<xacro:property name="axisLength" value="0.20321"/>
+	<xacro:property name="axisWidth" value="0.27070"/>
+	<xacro:property name="axisMass" value="20.0"/>
+	<xacro:property name="suspension_arm_F_Height" value="0.30536"/>
+	<xacro:property name="suspension_arm_F_Length" value="1.02203"/>
+	<xacro:property name="suspension_arm_F_Width" value="0.39606"/>
+	<xacro:property name="suspension_arm_F_Mass" value="20.0"/>
 	<!-- Differential-drive wheels properties -->
 	<xacro:property name="wheelWidth" value="0.026"/>

Commit message: Added trees and adding wheels

File: curiosity_mars_rover_description/urdf/chassis.xacro (robot description, xacro)
@@ -98,5 +98,5 @@
         <axis xyz="1 0 0"/>
 	</joint>
-	<link name='suspension_arm_B_L'>
+  	<link name='suspension_arm_B_L'>
 		<collision>
 			<origin xyz="0 0 0"
@@ -252,5 +252,5 @@
         <axis xyz="1 0 0"/>
 	</joint>
-	<link name='suspension_arm_B_R'>
+  	<link name='suspension_arm_B_R'>
 		<collision>
 			<origin xyz="0 0 0"

File: curiosity_mars_rover_description/urdf/curiosity_mars_rover.xacro (robot description, xacro)
@@ -9,10 +9,10 @@
 	<!-- Chasis -->
 	<xacro:include filename="$(find curiosity_mars_rover_description)/urdf/chassis.xacro" />
-	<!-- Arms -->
-	<!--
-	<xacro:include filename="$(find curiosity_mars_rover_description)/urdf/wheel_tree.xacro" />
-	<wheel lr="left" tY="-1"/>
-	<wheel lr="right" tY="1"/>
-	-->
+	<!-- Wheel Groups -->
+	<xacro:include filename="$(find curiosity_mars_rover_description)/urdf/wheel.xacro" />
+	<xacro:include filename="$(find curiosity_mars_rover_description)/urdf/left_wheel_group.xacro" />
+	<xacro:include filename="$(find curiosity_mars_rover_description)/urdf/right_wheel_group.xacro" />
 	<chassis_body/>
+	<left_wheel_tree/>
+	<right_wheel_tree/>
 </robot>

File: curiosity_mars_rover_description/urdf/curiosity_mars_rover_properties.xacro (robot description, xacro)
@@ -24,7 +24,6 @@
 	<xacro:property name="suspension_arm_F_Mass" value="20.0"/>
 	<!-- Differential-drive wheels properties -->
-	<xacro:property name="wheelWidth" value="0.026"/>
-	<xacro:property name="wheelRadius" value="0.032"/>
+	<xacro:property name="wheelWidth" value="0.39473"/>
+	<xacro:property name="wheelRadius" value="0.242645"/>
 	<xacro:property name="wheelMass" value="0.05"/>
-	<xacro:property name="wheelOffsetY" value="0.037"/>
 </robot>

File: curiosity_mars_rover_description/urdf/macros.xacro (robot description, xacro)
@@ -34,69 +34,3 @@
     />
   </xacro:macro>
-  <xacro:macro name="wheel" params="lr tY">
-    <link name="${lr}_wheel">
-      <collision>
-        <origin xyz="0 0 0"
-        		rpy="${-tY*PI/2} 0 0" />
-        <geometry>
-          <cylinder
-            length="${wheelWidth*scale_XYZ}"
-            radius="${wheelRadius*scale_XYZ}"/>
-        </geometry>
-      </collision>
-      <visual>
-        <origin xyz="0 0 0"
-        		rpy="${-tY*PI/2} 0 0" />
-        <geometry>
-          <mesh filename="package://garbagecollector_description/meshes/${lr}_wheel.dae" scale="${scale_XYZ} ${scale_XYZ} ${scale_XYZ}"/>
-        </geometry>
-      </visual>
-      <inertial>
-        <origin xyz="0 0 0"
-        		rpy="${-tY*PI/2} 0 0" />
-        <mass value="${wheelMass}"/>
-        <cylinder_inertia
-          m="${wheelMass}"
-          r="${wheelRadius*scale_XYZ}"
-          h="${wheelWidth*scale_XYZ}"/>
-      </inertial>
-    </link>
-    <gazebo reference="${lr}_wheel">
-      <mu1 value="1.0"/>
-      <mu2 value="1.0"/>
-      <kp  value="10000000.0" />
-      <kd>100.0</kd>
-      <minDepth>0.001</minDepth>
-      <maxVel>1.0</maxVel>
-      <!--kd  value="1.0" />
-      <fdir1 value="1 0 0"/-->
-      <material>Gazebo/FlatBlack</material>
-    </gazebo>
-    <joint name="${lr}_wheel_hinge" type="continuous">
-      <parent link="chassis"/>
-      <child link="${lr}_wheel"/>
-      <origin
-        xyz = "0 ${-tY*(wheelOffsetY+wheelWidth)*scale_XYZ} ${wheelRadius*scale_XYZ}"
-        rpy = "0 0 0" />
-      <axis xyz="0 1 0"
-      		  rpy="0 0 0" />
-      <!--limit effort="100" velocity="10"/-->
-      <limit effort="0.0" velocity="0.0"/>
-      <joint_properties damping="0.0" friction="0.0"/>
-    </joint>
-<!--
-  http://gazebosim.org/tutorials/?tut=ros_control
--->
-    <transmission name="${lr}_trans">
-      <type>transmission_interface/SimpleTransmission</type>
-      <joint name="${lr}_wheel_hinge">
-        <hardwareInterface>EffortJointInterface</hardwareInterface>
-      </joint>
-      <actuator name="${lr}Motor">
-        <hardwareInterface>EffortJointInterface</hardwareInterface>
-        <mechanicalReduction>10</mechanicalReduction>
-        <!--mechanicalReduction>1</mechanicalReduction-->
-      </actuator>
-    </transmission>
-  </xacro:macro>
 </robot>
