Commit message: Added all six wheels

File: curiosity_mars_rover_description/urdf/left_wheel_group.xacro (robot description, xacro)
@@ -60,4 +60,32 @@
         <axis xyz="0 0 1"/>
 	</joint>
+	<link name='suspension_steer_F_L_to_front_wheel_L'>
+		<inertial>
+            <origin xyz="0 0 0" rpy="0 0 0"/>
+            <mass value="0.02" />
+            <inertia ixx="2.61666666667e-05" ixy="0.0" ixz="0.0" iyy="2.61666666667e-05" iyz="0.0" izz="3.6e-05"/>
+        </inertial>
+        <collision>
+            <origin rpy="0.0 1.57 0" xyz="0 0 0"/>
+            <geometry>
+                <cylinder radius="0.02" length="0.02"/>
+            </geometry>
+        </collision>
+		<visual>
+            <origin rpy="0.0 1.57 0" xyz="0 0 0"/>
+            <geometry>
+                <cylinder radius="0.02" length="0.02"/>
+            </geometry>
+        </visual>
+	</link>
+	<joint name="suspension_steer_F_L_to_suspension_steer_F_L_to_front_wheel_L_joint" type="fixed">
+		<parent link="suspension_steer_F_L"/>
+		<child link="suspension_steer_F_L_to_front_wheel_L"/>
+		<origin xyz="0 0 -0.3996" rpy="0 0 0"/>
+	</joint>
+  	<wheel
+		wheel_name="front_wheel_L"
+		wheel_conector_name="suspension_steer_F_L_to_front_wheel_L"
+		tY="0"/>
   	<!-- FRONT LEFT Wheel Left END -->
 	<!-- MIDDLE WHEEL -->
@@ -71,11 +99,11 @@
             <origin rpy="0.0 1.57 0" xyz="0 0 0"/>
             <geometry>
-                <cylinder radius="0.242645" length="0.39473"/>
-            </geometry>
-        </collision>
-		<visual>
-            <origin rpy="0.0 1.57 0" xyz="0 0 0"/>
-            <geometry>
-                <cylinder radius="0.242645" length="0.39473"/>
+                <cylinder radius="0.02" length="0.02"/>
+            </geometry>
+        </collision>
+		<visual>
+            <origin rpy="0.0 1.57 0" xyz="0 0 0"/>
+            <geometry>
+                <cylinder radius="0.02" length="0.02"/>
             </geometry>
         </visual>
@@ -149,4 +177,32 @@
         <axis xyz="0 0 1"/>
 	</joint>
+  	<link name='suspension_steer_B_L_to_back_wheel_L'>
+		<inertial>
+            <origin xyz="0 0 0" rpy="0 0 0"/>
+            <mass value="0.02" />
+            <inertia ixx="2.61666666667e-05" ixy="0.0" ixz="0.0" iyy="2.61666666667e-05" iyz="0.0" izz="3.6e-05"/>
+        </inertial>
+        <collision>
+            <origin rpy="0.0 1.57 0" xyz="0 0 0"/>
+            <geometry>
+                <cylinder radius="0.02" length="0.02"/>
+            </geometry>
+        </collision>
+		<visual>
+            <origin rpy="0.0 1.57 0" xyz="0 0 0"/>
+            <geometry>
+                <cylinder radius="0.02" length="0.02"/>
+            </geometry>
+        </visual>
+	</link>
+	<joint name="suspension_arm_B2_L_to_suspension_steer_B_L_to_back_wheel_L_joint" type="fixed">
+		<parent link="suspension_steer_B_L"/>
+		<child link="suspension_steer_B_L_to_back_wheel_L"/>
+		<origin xyz="0 0 -0.410523" rpy="0 0 0"/>
+	</joint>
+  	<wheel
+		wheel_name="back_wheel_L"
+		wheel_conector_name="suspension_steer_B_L_to_back_wheel_L"
+		tY="0"/>
   	<!-- END BACK WHEEL LEFT -->
   </xacro:macro>

File: curiosity_mars_rover_description/urdf/right_wheel_group.xacro (robot description, xacro)
@@ -60,5 +60,61 @@
         <axis xyz="0 0 1"/>
 	</joint>
+	<link name='suspension_steer_F_R_to_front_wheel_R'>
+		<inertial>
+            <origin xyz="0 0 0" rpy="0 0 0"/>
+            <mass value="0.02" />
+            <inertia ixx="2.61666666667e-05" ixy="0.0" ixz="0.0" iyy="2.61666666667e-05" iyz="0.0" izz="3.6e-05"/>
+        </inertial>
+        <collision>
+            <origin rpy="0.0 1.57 0" xyz="0 0 0"/>
+            <geometry>
+                <cylinder radius="0.02" length="0.02"/>
+            </geometry>
+        </collision>
+		<visual>
+            <origin rpy="0.0 1.57 0" xyz="0 0 0"/>
+            <geometry>
+                <cylinder radius="0.02" length="0.02"/>
+            </geometry>
+        </visual>
+	</link>
+	<joint name="suspension_steer_F_R_to_suspension_steer_F_R_to_front_wheel_R_joint" type="fixed">
+		<parent link="suspension_steer_F_R"/>
+		<child link="suspension_steer_F_R_to_front_wheel_R"/>
+		<origin xyz="0 0 -0.3996" rpy="0 0 0"/>
+	</joint>
+  	<wheel
+		wheel_name="front_wheel_R"
+		wheel_conector_name="suspension_steer_F_R_to_front_wheel_R"
+		tY="-1"/>
   	<!-- FRONT WHEEL RIGHT END -->
+	<link name='suspension_arm_B2_R_to_middle_wheel_R'>
+		<inertial>
+            <origin xyz="0 0 0" rpy="0 0 0"/>
+            <mass value="0.02" />
+            <inertia ixx="2.61666666667e-05" ixy="0.0" ixz="0.0" iyy="2.61666666667e-05" iyz="0.0" izz="3.6e-05"/>
+        </inertial>
+        <collision>
+            <origin rpy="0.0 1.57 0" xyz="0 0 0"/>
+            <geometry>
+                <cylinder radius="0.02" length="0.02"/>
+            </geometry>
+        </collision>
+		<visual>
+            <origin rpy="0.0 1.57 0" xyz="0 0 0"/>
+            <geometry>
+                <cylinder radius="0.02" length="0.02"/>
+            </geometry>
+        </visual>
+	</link>
+	<joint name="suspension_arm_B2_R_to_suspension_arm_B2_R_to_middle_wheel_R_joint" type="fixed">
+		<parent link="suspension_arm_B2_R"/>
+		<child link="suspension_arm_B2_R_to_middle_wheel_R"/>
+		<origin xyz="-0.39423 -0.44859 -0.41098" rpy="0 0 0"/>
+	</joint>
+  	<wheel
+		wheel_name="middle_wheel_R"
+		wheel_conector_name="suspension_arm_B2_R_to_middle_wheel_R"
+		tY="-1"/>
   	<!-- RIGHT BACK WHEEL -->
 	<link name='suspension_arm_B2_R_to_suspension_steer_B_R'>
@@ -119,4 +175,32 @@
         <axis xyz="0 0 1"/>
 	</joint>
+	<link name='suspension_steer_B_R_to_back_wheel_R'>
+		<inertial>
+            <origin xyz="0 0 0" rpy="0 0 0"/>
+            <mass value="0.02" />
+            <inertia ixx="2.61666666667e-05" ixy="0.0" ixz="0.0" iyy="2.61666666667e-05" iyz="0.0" izz="3.6e-05"/>
+        </inertial>
+        <collision>
+            <origin rpy="0.0 1.57 0" xyz="0 0 0"/>
+            <geometry>
+                <cylinder radius="0.02" length="0.02"/>
+            </geometry>
+        </collision>
+		<visual>
+            <origin rpy="0.0 1.57 0" xyz="0 0 0"/>
+            <geometry>
+                <cylinder radius="0.02" length="0.02"/>
+            </geometry>
+        </visual>
+	</link>
+	<joint name="suspension_arm_B2_R_to_suspension_steer_B_R_to_back_wheel_R_joint" type="fixed">
+		<parent link="suspension_steer_B_R"/>
+		<child link="suspension_steer_B_R_to_back_wheel_R"/>
+		<origin xyz="0 0 -0.410523" rpy="0 0 0"/>
+	</joint>
+  	<wheel
+		wheel_name="back_wheel_R"
+		wheel_conector_name="suspension_steer_B_R_to_back_wheel_R"
+		tY="-1"/>
   	<!-- END BACK WHEEL RIGHT -->
   </xacro:macro>

File: curiosity_mars_rover_description/urdf/wheel.xacro (robot description, xacro)
@@ -43,5 +43,5 @@
 		<origin xyz="0 0 0" rpy="0 0 ${tY*PI}"/>
 		<limit effort="10000.0" velocity="100.0"/>
-        <axis xyz="0 0 1"/>
+        <axis xyz="1 0 0"/>
         <joint_properties damping="0.0" friction="0.0"/>
 	</joint>
