Commit message: Added arm and adding sensor mast

File: curiosity_mars_rover_description/urdf/curiosity_mars_rover.xacro (robot description, xacro)
@@ -13,6 +13,12 @@
 	<xacro:include filename="$(find curiosity_mars_rover_description)/urdf/left_wheel_group.xacro" />
 	<xacro:include filename="$(find curiosity_mars_rover_description)/urdf/right_wheel_group.xacro" />
+	<!-- Arm -->
+	<xacro:include filename="$(find curiosity_mars_rover_description)/urdf/arm.xacro" />
+	<!-- Sensor Mast -->
+	<xacro:include filename="$(find curiosity_mars_rover_description)/urdf/sensor_mast.xacro" />
 	<chassis_body/>
 	<left_wheel_tree/>
 	<right_wheel_tree/>
+	<arm/>
+	<sensor_mast/>
 </robot>

File: curiosity_mars_rover_description/urdf/curiosity_mars_rover_properties.xacro (robot description, xacro)
@@ -23,4 +23,8 @@
 	<xacro:property name="suspension_arm_F_Width" value="0.39606"/>
 	<xacro:property name="suspension_arm_F_Mass" value="20.0"/>
+	<xacro:property name="armHeight" value="0.01"/>
+	<xacro:property name="armLength" value="0.01"/>
+	<xacro:property name="armWidth" value="0.01"/>
+	<xacro:property name="armMass" value="0.01"/>
 	<!-- Differential-drive wheels properties -->
 	<xacro:property name="wheelWidth" value="0.39473"/>
