Commit message: Added improvement in the wheels

File: curiosity_mars_rover_description/urdf/curiosity_mars_rover_properties.xacro (robot description, xacro)
@@ -21,12 +21,16 @@
 	<xacro:property name="suspension_arm_F_L_Y" value="1.02203"/>
 	<xacro:property name="suspension_arm_F_L_Z" value="0.30536"/>
+	<xacro:property name="suspension_arm_F_L_limit" value="0.4"/>
 	<xacro:property name="suspension_arm_B_L_Mass" value="${TreeMass/TreeParts}"/>
 	<xacro:property name="suspension_arm_B_L_X" value="0.123524"/>
 	<xacro:property name="suspension_arm_B_L_Y" value="0.852108"/>
 	<xacro:property name="suspension_arm_B_L_Z" value="0.348354"/>
+	<xacro:property name="suspension_arm_B_L_limit" value="0.4"/>
 	<xacro:property name="suspension_arm_B2_L_Mass" value="${TreeMass/TreeParts}"/>
 	<xacro:property name="suspension_arm_B2_L_X" value="0.400262"/>
 	<xacro:property name="suspension_arm_B2_L_Y" value="1.22113"/>
 	<xacro:property name="suspension_arm_B2_L_Z" value="0.631338"/>
+	<xacro:property name="suspension_arm_B2_lower_limit" value="-1.2"/>
+	<xacro:property name="suspension_arm_B2_upper_limit" value="0.1"/>
 	<xacro:property name="suspension_steer_F_L_Mass" value="${TreeMass/TreeParts}"/>
 	<xacro:property name="suspension_steer_F_L_X" value="0.528399"/>
@@ -37,7 +41,14 @@
 	<xacro:property name="suspension_steer_B_L_Y" value="0.21019"/>
 	<xacro:property name="suspension_steer_B_L_Z" value="0.450036"/>
+	<xacro:property name="suspension_steer_limit" value="0.6"/>
+	<xacro:property name="suspension_steer_effort" value="10000.0"/>
+	<xacro:property name="suspension_steer_velocity" value="10.0"/>
+	<xacro:property name="suspension_effort" value="10000.0"/>
+	<xacro:property name="suspension_speed" value="10.0"/>
+	<xacro:property name="suspension_damping" value="0.5"/>
+	<xacro:property name="suspension_friction" value="0.5"/>
 	<!-- Wheels properties -->
 	<xacro:property name="wheelWidth" value="0.39473"/>
-	<xacro:property name="wheelRadius" value="0.242645"/>
+	<xacro:property name="wheelRadius" value="0.242647"/>
 	<xacro:property name="wheelMass" value="2.07"/>
 	<!-- Arm -->

File: curiosity_mars_rover_description/urdf/left_wheel_group.xacro (robot description, xacro)
@@ -63,7 +63,18 @@
 		<child link="suspension_arm_F_L"/>
 		<origin xyz="0 0 0" rpy="0 0 0"/>
-		<limit lower="-0.2" upper="0.2" effort="10000.0" velocity="100.0"/>
+		<limit lower="${-suspension_arm_F_L_limit}" upper="${suspension_arm_F_L_limit}" effort="${suspension_effort}" velocity="${suspension_speed}"/>
         <axis xyz="1 0 0"/>
-	</joint>
+		<joint_properties damping="${suspension_damping}" friction="${suspension_friction}"/>
+	</joint>
+	<transmission name="suspension_arm_F_L_trans">
+      <type>transmission_interface/SimpleTransmission</type>
+      <joint name="suspension_arm_F_L_joint">
+        <hardwareInterface>hardware_interface/EffortJointInterface</hardwareInterface>
+      </joint>
+      <actuator name="suspension_arm_F_LMotor">
+        <hardwareInterface>hardware_interface/EffortJointInterface</hardwareInterface>
+        <mechanicalReduction>1</mechanicalReduction>
+      </actuator>
+    </transmission>
   	<link name='suspension_arm_B_L'>
 		<collision>
@@ -96,7 +107,18 @@
 		<child link="suspension_arm_B_L"/>
 		<origin xyz="0 0 0" rpy="0 0 0"/>
-		<limit lower="-0.2" upper="0.2" effort="10000.0" velocity="100.0"/>
+		<limit lower="${-suspension_arm_B_L_limit}" upper="${suspension_arm_B_L_limit}" effort="${suspension_effort}" velocity="${suspension_speed}"/>
         <axis xyz="1 0 0"/>
-	</joint>
+		<joint_properties damping="${suspension_damping}" friction="${suspension_friction}"/>
+	</joint>
+	<transmission name="suspension_arm_B_L_trans">
+      <type>transmission_interface/SimpleTransmission</type>
+      <joint name="suspension_arm_B_L_joint">
+        <hardwareInterface>hardware_interface/EffortJointInterface</hardwareInterface>
+      </joint>
+      <actuator name="suspension_arm_B_LMotor">
+        <hardwareInterface>hardware_interface/EffortJointInterface</hardwareInterface>
+        <mechanicalReduction>1</mechanicalReduction>
+      </actuator>
+    </transmission>
  	<link name='suspension_arm_B_L_to_B2_L'>
 		<inertial>
@@ -153,7 +175,18 @@
 		<child link="suspension_arm_B2_L"/>
 		<origin xyz="0 0 0" rpy="0 0 0"/>
-		<limit lower="-0.2" upper="0.2" effort="10000.0" velocity="100.0"/>
+		<limit lower="${suspension_arm_B2_lower_limit}" upper="${suspension_arm_B2_upper_limit}" effort="${suspension_effort}" velocity="${suspension_speed}"/>
         <axis xyz="1 0 0"/>
-	</joint>
+		<joint_properties damping="${suspension_damping}" friction="${suspension_friction}"/>
+	</joint>
+	<transmission name="suspension_arm_B2_L_trans">
+      <type>transmission_interface/SimpleTransmission</type>
+      <joint name="suspension_arm_B2_L_joint">
+        <hardwareInterface>hardware_interface/EffortJointInterface</hardwareInterface>
+      </joint>
+      <actuator name="suspension_arm_B2_LMotor">
+        <hardwareInterface>hardware_interface/EffortJointInterface</hardwareInterface>
+        <mechanicalReduction>1</mechanicalReduction>
+      </actuator>
+    </transmission>
 	<!-- FRONT WHEEL -->
 	<link name='suspension_arm_F_L_to_suspension_steer_F_L'>
@@ -211,7 +244,17 @@
 		<child link="suspension_steer_F_L"/>
 		<origin xyz="0 0 0" rpy="0 0 0"/>
-		<limit lower="-0.2" upper="0.2" effort="10000.0" velocity="100.0"/>
+		<limit lower="${-suspension_steer_limit}" upper="${suspension_steer_limit}" effort="${suspension_steer_effort}" velocity="${suspension_steer_velocity}"/>
         <axis xyz="0 0 1"/>
 	</joint>
+	<transmission name="suspension_steer_F_L_trans">
+      <type>transmission_interface/SimpleTransmission</type>
+      <joint name="suspension_steer_F_L_joint">
+        <hardwareInterface>hardware_interface/EffortJointInterface</hardwareInterface>
+      </joint>
+      <actuator name="suspension_steer_F_LMotor">
+        <hardwareInterface>hardware_interface/EffortJointInterface</hardwareInterface>
+        <mechanicalReduction>1</mechanicalReduction>
+      </actuator>
+    </transmission>
 	<link name='suspension_steer_F_L_to_front_wheel_L'>
 		<inertial>
@@ -328,7 +371,17 @@
 		<child link="suspension_steer_B_L"/>
 		<origin xyz="0 0 0" rpy="0 0 0"/>
-		<limit lower="-0.2" upper="0.2" effort="10000.0" velocity="100.0"/>
+		<limit lower="${-suspension_steer_limit}" upper="${suspension_steer_limit}" effort="${suspension_steer_effort}" velocity="${suspension_steer_velocity}"/>
         <axis xyz="0 0 1"/>
 	</joint>
+	<transmission name="suspension_steer_B_L_trans">
+      <type>transmission_interface/SimpleTransmission</type>
+      <joint name="suspension_steer_B_L_joint">
+        <hardwareInterface>hardware_interface/EffortJointInterface</hardwareInterface>
+      </joint>
+      <actuator name="suspension_steer_B_LMotor">
+        <hardwareInterface>hardware_interface/EffortJointInterface</hardwareInterface>
+        <mechanicalReduction>1</mechanicalReduction>
+      </actuator>
+    </transmission>
   	<link name='suspension_steer_B_L_to_back_wheel_L'>
 		<inertial>

File: curiosity_mars_rover_description/urdf/right_wheel_group.xacro (robot description, xacro)
@@ -63,7 +63,18 @@
 		<child link="suspension_arm_F_R"/>
 		<origin xyz="0 0 0" rpy="0 0 0"/>
-		<limit lower="-0.2" upper="0.2" effort="10000.0" velocity="100.0"/>
+		<limit lower="${-suspension_arm_F_L_limit}" upper="${suspension_arm_F_L_limit}" effort="${suspension_effort}" velocity="${suspension_speed}"/>
         <axis xyz="1 0 0"/>
-	</joint>
+		<joint_properties damping="${suspension_damping}" friction="${suspension_friction}"/>
+	</joint>
+  	<transmission name="suspension_arm_F_R_trans">
+      <type>transmission_interface/SimpleTransmission</type>
+      <joint name="suspension_arm_F_R_joint">
+        <hardwareInterface>hardware_interface/EffortJointInterface</hardwareInterface>
+      </joint>
+      <actuator name="suspension_arm_F_RMotor">
+        <hardwareInterface>hardware_interface/EffortJointInterface</hardwareInterface>
+        <mechanicalReduction>1</mechanicalReduction>
+      </actuator>
+    </transmission>
   	<link name='suspension_arm_B_R'>
 		<collision>
@@ -96,7 +107,18 @@
 		<child link="suspension_arm_B_R"/>
 		<origin xyz="0 0 0" rpy="0 0 0"/>
-		<limit lower="-0.2" upper="0.2" effort="10000.0" velocity="100.0"/>
+		<limit lower="${-suspension_arm_B_L_limit}" upper="${suspension_arm_B_L_limit}" effort="${suspension_effort}" velocity="${suspension_speed}"/>
         <axis xyz="1 0 0"/>
-	</joint>
+		<joint_properties damping="${suspension_damping}" friction="${suspension_friction}"/>
+	</joint>
+  	<transmission name="suspension_arm_B_R_trans">
+      <type>transmission_interface/SimpleTransmission</type>
+      <joint name="suspension_arm_B_R_joint">
+        <hardwareInterface>hardware_interface/EffortJointInterface</hardwareInterface>
+      </joint>
+      <actuator name="suspension_arm_B_RMotor">
+        <hardwareInterface>hardware_interface/EffortJointInterface</hardwareInterface>
+        <mechanicalReduction>1</mechanicalReduction>
+      </actuator>
+    </transmission>
   	<link name='suspension_arm_B_R_to_B2_R'>
 		<inertial>
@@ -153,7 +175,18 @@
 		<child link="suspension_arm_B2_R"/>
 		<origin xyz="0 0 0" rpy="0 0 0"/>
-		<limit lower="-0.2" upper="0.2" effort="10000.0" velocity="100.0"/>
+		<limit lower="${suspension_arm_B2_lower_limit}" upper="${suspension_arm_B2_upper_limit}" effort="${suspension_effort}" velocity="${suspension_speed}"/>
         <axis xyz="1 0 0"/>
-	</joint>
+		<joint_properties damping="${suspension_damping}" friction="${suspension_friction}"/>
+	</joint>
+  	<transmission name="suspension_arm_B2_R_trans">
+      <type>transmission_interface/SimpleTransmission</type>
+      <joint name="suspension_arm_B2_R_joint">
+        <hardwareInterface>hardware_interface/EffortJointInterface</hardwareInterface>
+      </joint>
+      <actuator name="suspension_arm_B2_RMotor">
+        <hardwareInterface>hardware_interface/EffortJointInterface</hardwareInterface>
+        <mechanicalReduction>1</mechanicalReduction>
+      </actuator>
+    </transmission>
 	<!-- FRONT WHEEL RIGHT -->
 	<link name='suspension_arm_F_R_to_suspension_steer_F_R'>
@@ -211,7 +244,17 @@
 		<child link="suspension_steer_F_R"/>
 		<origin xyz="0 0 0" rpy="0 0 0"/>
-		<limit lower="-0.2" upper="0.2" effort="10000.0" velocity="100.0"/>
+		<limit lower="${-suspension_steer_limit}" upper="${suspension_steer_limit}" effort="${suspension_steer_effort}" velocity="${suspension_steer_velocity}"/>
         <axis xyz="0 0 1"/>
 	</joint>
+	<transmission name="suspension_steer_F_R_trans">
+      <type>transmission_interface/SimpleTransmission</type>
+      <joint name="suspension_steer_F_R_joint">
+        <hardwareInterface>hardware_interface/EffortJointInterface</hardwareInterface>
+      </joint>
+      <actuator name="suspension_steer_F_RMotor">
+        <hardwareInterface>hardware_interface/EffortJointInterface</hardwareInterface>
+        <mechanicalReduction>1</mechanicalReduction>
+      </actuator>
+    </transmission>
 	<link name='suspension_steer_F_R_to_front_wheel_R'>
 		<inertial>
@@ -326,7 +369,17 @@
 		<child link="suspension_steer_B_R"/>
 		<origin xyz="0 0 0" rpy="0 0 0"/>
-		<limit lower="-0.2" upper="0.2" effort="10000.0" velocity="100.0"/>
+		<limit lower="${-suspension_steer_limit}" upper="${suspension_steer_limit}" effort="${suspension_steer_effort}" velocity="${suspension_steer_velocity}"/>
         <axis xyz="0 0 1"/>
 	</joint>
+  	<transmission name="suspension_steer_B_R_trans">
+      <type>transmission_interface/SimpleTransmission</type>
+      <joint name="suspension_steer_B_R_joint">
+        <hardwareInterface>hardware_interface/EffortJointInterface</hardwareInterface>
+      </joint>
+      <actuator name="suspension_steer_B_RMotor">
+        <hardwareInterface>hardware_interface/EffortJointInterface</hardwareInterface>
+        <mechanicalReduction>1</mechanicalReduction>
+      </actuator>
+    </transmission>
 	<link name='suspension_steer_B_R_to_back_wheel_R'>
 		<inertial>

File: curiosity_mars_rover_description/urdf/wheel.xacro (robot description, xacro)
@@ -6,7 +6,7 @@
 		<collision>
 			<origin xyz="0 0 0"
-					rpy="0 0 0"/>
+					rpy="0 1.57 0"/>
 			<geometry>
-				<mesh filename="package://curiosity_mars_rover_description/meshes/wheel.dae" scale="${scale_XYZ} ${scale_XYZ} ${scale_XYZ}"/>
+				<cylinder radius="${wheelRadius}" length="${wheelWidth}"/>
 			</geometry>
 		</collision>
@@ -15,5 +15,5 @@
 					rpy="0 0 0"/>
 			<geometry>
-				<mesh filename="package://curiosity_mars_rover_description/meshes/wheel.dae" scale="${scale_XYZ} ${scale_XYZ} ${scale_XYZ}"/>
+				<mesh filename="package://curiosity_mars_rover_description/meshes/wheel_fixed.dae" scale="${scale_XYZ} ${scale_XYZ} ${scale_XYZ}"/>
 			</geometry>
 		</visual>
