Commit message: Added correct innertias and masses

File: curiosity_mars_rover_description/urdf/arm.xacro (robot description, xacro)
@@ -44,10 +44,10 @@
 			<origin xyz="0 0 0"
 					rpy="0 0 0"/>
-			<mass value="${armMass}"/>
-			<box_inertia
-				m="${armMass}"
-				x="${armWidth*scale_XYZ}"
-				y="${armLength*scale_XYZ}"
-				z="${armHeight*scale_XYZ}"/>
+			<mass value="${arm_01_Mass}"/>
+			<box_inertia
+				m="${arm_01_Mass}"
+				x="${arm_01_X*scale_XYZ}"
+				y="${arm_01_Y*scale_XYZ}"
+				z="${arm_01_Z*scale_XYZ}"/>
 		</inertial>
 	</link>
@@ -112,10 +112,10 @@
 			<origin xyz="0 0 0"
 					rpy="0 0 0"/>
-			<mass value="${armMass}"/>
-			<box_inertia
-				m="${armMass}"
-				x="${armWidth*scale_XYZ}"
-				y="${armLength*scale_XYZ}"
-				z="${armHeight*scale_XYZ}"/>
+			<mass value="${arm_02_Mass}"/>
+			<box_inertia
+				m="${arm_02_Mass}"
+				x="${arm_02_X*scale_XYZ}"
+				y="${arm_02_Y*scale_XYZ}"
+				z="${arm_02_Z*scale_XYZ}"/>
 		</inertial>
 	</link>
@@ -180,10 +180,10 @@
 			<origin xyz="0 0 0"
 					rpy="0 0 0"/>
-			<mass value="${armMass}"/>
-			<box_inertia
-				m="${armMass}"
-				x="${armWidth*scale_XYZ}"
-				y="${armLength*scale_XYZ}"
-				z="${armHeight*scale_XYZ}"/>
+			<mass value="${arm_03_Mass}"/>
+			<box_inertia
+				m="${arm_03_Mass}"
+				x="${arm_03_X*scale_XYZ}"
+				y="${arm_03_Y*scale_XYZ}"
+				z="${arm_03_Z*scale_XYZ}"/>
 		</inertial>
 	</link>
@@ -248,10 +248,10 @@
 			<origin xyz="0 0 0"
 					rpy="0 0 0"/>
-			<mass value="${armMass}"/>
-			<box_inertia
-				m="${armMass}"
-				x="${armWidth*scale_XYZ}"
-				y="${armLength*scale_XYZ}"
-				z="${armHeight*scale_XYZ}"/>
+			<mass value="${arm_04_Mass}"/>
+			<box_inertia
+				m="${arm_04_Mass}"
+				x="${arm_04_X*scale_XYZ}"
+				y="${arm_04_Y*scale_XYZ}"
+				z="${arm_04_Z*scale_XYZ}"/>
 		</inertial>
 	</link>
@@ -316,10 +316,10 @@
 			<origin xyz="0 0 0"
 					rpy="0 0 0"/>
-			<mass value="${armMass}"/>
-			<box_inertia
-				m="${armMass}"
-				x="${armWidth*scale_XYZ}"
-				y="${armLength*scale_XYZ}"
-				z="${armHeight*scale_XYZ}"/>
+			<mass value="${arm_tools_Mass}"/>
+			<box_inertia
+				m="${arm_tools_Mass}"
+				x="${arm_tools_X*scale_XYZ}"
+				y="${arm_tools_Y*scale_XYZ}"
+				z="${arm_tools_Z*scale_XYZ}"/>
 		</inertial>
 	</link>

File: curiosity_mars_rover_description/urdf/chassis.xacro (robot description, xacro)
@@ -34,312 +34,4 @@
 		</inertial>
 	</link>
-  	<link name='left_axis'>
-		<collision>
-			<origin xyz="0 0 0"
-					rpy="0 0 0"/>
-			<geometry>
-				<mesh filename="package://curiosity_mars_rover_description/meshes/left_axis_jointfix_v2.dae" scale="${scale_XYZ} ${scale_XYZ} ${scale_XYZ}"/>
-			</geometry>
-		</collision>
-		<visual>
-			<origin xyz="0 0 0"
-					rpy="0 0 0"/>
-			<geometry>
-				<mesh filename="package://curiosity_mars_rover_description/meshes/left_axis_jointfix_v2.dae" scale="${scale_XYZ} ${scale_XYZ} ${scale_XYZ}"/>
-			</geometry>
-		</visual>
-		<inertial>
-			<origin xyz="0 0 0"
-					rpy="0 0 0"/>
-			<mass value="${axisMass}"/>
-			<box_inertia
-				m="${axisMass}"
-				x="${axisWidth*scale_XYZ}"
-				y="${axisLength*scale_XYZ}"
-				z="${axisHeight*scale_XYZ}"/>
-		</inertial>
-	</link>
-  	<joint name="left_axis_joint" type="fixed">
-		<parent link="chassis"/>
-		<child link="left_axis"/>
-		<origin xyz="0.7938 -0.2133 0" rpy="0 -0.19565141 0"/>
-	</joint>
-  	<link name='suspension_arm_F_L'>
-		<collision>
-			<origin xyz="0 0 0"
-					rpy="0 0 0"/>
-			<geometry>
-				<mesh filename="package://curiosity_mars_rover_description/meshes/suspension_arm_F_L_fixed.dae" scale="${scale_XYZ} ${scale_XYZ} ${scale_XYZ}"/>
-			</geometry>
-		</collision>
-		<visual>
-			<origin xyz="0 0 0"
-					rpy="0 0 0"/>
-			<geometry>
-				<mesh filename="package://curiosity_mars_rover_description/meshes/suspension_arm_F_L_fixed.dae" scale="${scale_XYZ} ${scale_XYZ} ${scale_XYZ}"/>
-			</geometry>
-		</visual>
-		<inertial>
-			<origin xyz="0 0 0"
-					rpy="0 0 0"/>
-			<mass value="${suspension_arm_F_Mass}"/>
-			<box_inertia
-				m="${suspension_arm_F_Mass}"
-				x="${suspension_arm_F_Width*scale_XYZ}"
-				y="${suspension_arm_F_Length*scale_XYZ}"
-				z="${suspension_arm_F_Height*scale_XYZ}"/>
-		</inertial>
-	</link>
-  	<joint name="suspension_arm_F_L_joint" type="revolute">
-		<parent link="left_axis"/>
-		<child link="suspension_arm_F_L"/>
-		<origin xyz="0 0 0" rpy="0 0 0"/>
-		<limit lower="-0.2" upper="0.2" effort="10000.0" velocity="100.0"/>
-        <axis xyz="1 0 0"/>
-	</joint>
-  	<link name='suspension_arm_B_L'>
-		<collision>
-			<origin xyz="0 0 0"
-					rpy="0 0 0"/>
-			<geometry>
-				<mesh filename="package://curiosity_mars_rover_description/meshes/suspension_arm_B_L_fixed.dae" scale="${scale_XYZ} ${scale_XYZ} ${scale_XYZ}"/>
-			</geometry>
-		</collision>
-		<visual>
-			<origin xyz="0 0 0"
-					rpy="0 0 0"/>
-			<geometry>
-				<mesh filename="package://curiosity_mars_rover_description/meshes/suspension_arm_B_L_fixed.dae" scale="${scale_XYZ} ${scale_XYZ} ${scale_XYZ}"/>
-			</geometry>
-		</visual>
-		<inertial>
-			<origin xyz="0 0 0"
-					rpy="0 0 0"/>
-			<mass value="${suspension_arm_F_Mass}"/>
-			<box_inertia
-				m="${suspension_arm_F_Mass}"
-				x="${suspension_arm_F_Width*scale_XYZ}"
-				y="${suspension_arm_F_Length*scale_XYZ}"
-				z="${suspension_arm_F_Height*scale_XYZ}"/>
-		</inertial>
-	</link>
-  	<joint name="suspension_arm_B_L_joint" type="revolute">
-		<parent link="left_axis"/>
-		<child link="suspension_arm_B_L"/>
-		<origin xyz="0 0 0" rpy="0 0 0"/>
-		<limit lower="-0.2" upper="0.2" effort="10000.0" velocity="100.0"/>
-        <axis xyz="1 0 0"/>
-	</joint>
- 	<link name='suspension_arm_B_L_to_B2_L'>
-		<inertial>
-            <origin xyz="0 0 0" rpy="0 0 0"/>
-            <mass value="0.02" />
-            <inertia ixx="2.61666666667e-05" ixy="0.0" ixz="0.0" iyy="2.61666666667e-05" iyz="0.0" izz="3.6e-05"/>
-        </inertial>
-        <collision>
-            <origin xyz="0 0 0.015" rpy="0 0 0"/>
-            <geometry>
-                <cylinder radius="0.06" length="0.035"/>
-            </geometry>
-        </collision>
-		<visual>
-            <origin rpy="0.0 1.57 0" xyz="0 0 0"/>
-            <geometry>
-                <cylinder radius="0.04" length="0.1"/>
-            </geometry>
-        </visual>
-	</link>
-	<joint name="suspension_arm_B_L_to_B2_L_joint" type="fixed">
-		<parent link="suspension_arm_B_L"/>
-		<child link="suspension_arm_B_L_to_B2_L"/>
-		<origin xyz="-0.05159 0.73683 -0.22972" rpy="0 0.1937315 0"/>
-	</joint>
-	<link name='suspension_arm_B2_L'>
-		<collision>
-			<origin xyz="0 0 0"
-					rpy="0 0 0"/>
-			<geometry>
-				<mesh filename="package://curiosity_mars_rover_description/meshes/suspension_arm_B2_L_fixed.dae" scale="${scale_XYZ} ${scale_XYZ} ${scale_XYZ}"/>
-			</geometry>
-		</collision>
-		<visual>
-			<origin xyz="0 0 0"
-					rpy="0 0 0"/>
-			<geometry>
-				<mesh filename="package://curiosity_mars_rover_description/meshes/suspension_arm_B2_L_fixed.dae" scale="${scale_XYZ} ${scale_XYZ} ${scale_XYZ}"/>
-			</geometry>
-		</visual>
-		<inertial>
-			<origin xyz="0 0 0"
-					rpy="0 0 0"/>
-			<mass value="${suspension_arm_F_Mass}"/>
-			<box_inertia
-				m="${suspension_arm_F_Mass}"
-				x="${suspension_arm_F_Width*scale_XYZ}"
-				y="${suspension_arm_F_Length*scale_XYZ}"
-				z="${suspension_arm_F_Height*scale_XYZ}"/>
-		</inertial>
-	</link>
-  	<joint name="suspension_arm_B2_L_joint" type="revolute">
-		<parent link="suspension_arm_B_L_to_B2_L"/>
-		<child link="suspension_arm_B2_L"/>
-		<origin xyz="0 0 0" rpy="0 0 0"/>
-		<limit lower="-0.2" upper="0.2" effort="10000.0" velocity="100.0"/>
-        <axis xyz="1 0 0"/>
-	</joint>
-  	<link name='right_axis'>
-		<collision>
-			<origin xyz="0 0 0"
-					rpy="0 0 0"/>
-			<geometry>
-				<mesh filename="package://curiosity_mars_rover_description/meshes/right_axis_jointfix_v2.dae" scale="${scale_XYZ} ${scale_XYZ} ${scale_XYZ}"/>
-			</geometry>
-		</collision>
-		<visual>
-			<origin xyz="0 0 0"
-					rpy="0 0 0"/>
-			<geometry>
-				<mesh filename="package://curiosity_mars_rover_description/meshes/right_axis_jointfix_v2.dae" scale="${scale_XYZ} ${scale_XYZ} ${scale_XYZ}"/>
-			</geometry>
-		</visual>
-		<inertial>
-			<origin xyz="0 0 0"
-					rpy="0 0 0"/>
-			<mass value="${axisMass}"/>
-			<box_inertia
-				m="${axisMass}"
-				x="${axisWidth*scale_XYZ}"
-				y="${axisLength*scale_XYZ}"
-				z="${axisHeight*scale_XYZ}"/>
-		</inertial>
-	</link>
-  	<joint name="right_axis_joint" type="fixed">
-		<parent link="chassis"/>
-		<child link="right_axis"/>
-		<origin xyz="-0.7938 -0.2133 0" rpy="0 0.19565141 0"/>
-	</joint>
-	<link name='suspension_arm_F_R'>
-		<collision>
-			<origin xyz="0 0 0"
-					rpy="0 0 0"/>
-			<geometry>
-				<mesh filename="package://curiosity_mars_rover_description/meshes/suspension_arm_F_R_fixed.dae" scale="${scale_XYZ} ${scale_XYZ} ${scale_XYZ}"/>
-			</geometry>
-		</collision>
-		<visual>
-			<origin xyz="0 0 0"
-					rpy="0 0 0"/>
-			<geometry>
-				<mesh filename="package://curiosity_mars_rover_description/meshes/suspension_arm_F_R_fixed.dae" scale="${scale_XYZ} ${scale_XYZ} ${scale_XYZ}"/>
-			</geometry>
-		</visual>
-		<inertial>
-			<origin xyz="0 0 0"
-					rpy="0 0 0"/>
-			<mass value="${suspension_arm_F_Mass}"/>
-			<box_inertia
-				m="${suspension_arm_F_Mass}"
-				x="${suspension_arm_F_Width*scale_XYZ}"
-				y="${suspension_arm_F_Length*scale_XYZ}"
-				z="${suspension_arm_F_Height*scale_XYZ}"/>
-		</inertial>
-	</link>
-  	<joint name="suspension_arm_F_R_joint" type="revolute">
-		<parent link="right_axis"/>
-		<child link="suspension_arm_F_R"/>
-		<origin xyz="0 0 0" rpy="0 0 0"/>
-		<limit lower="-0.2" upper="0.2" effort="10000.0" velocity="100.0"/>
-        <axis xyz="1 0 0"/>
-	</joint>
-  	<link name='suspension_arm_B_R'>
-		<collision>
-			<origin xyz="0 0 0"
-					rpy="0 0 0"/>
-			<geometry>
-				<mesh filename="package://curiosity_mars_rover_description/meshes/suspension_arm_B_R_fixed.dae" scale="${scale_XYZ} ${scale_XYZ} ${scale_XYZ}"/>
-			</geometry>
-		</collision>
-		<visual>
-			<origin xyz="0 0 0"
-					rpy="0 0 0"/>
-			<geometry>
-				<mesh filename="package://curiosity_mars_rover_description/meshes/suspension_arm_B_R_fixed.dae" scale="${scale_XYZ} ${scale_XYZ} ${scale_XYZ}"/>
-			</geometry>
-		</visual>
-		<inertial>
-			<origin xyz="0 0 0"
-					rpy="0 0 0"/>
-			<mass value="${suspension_arm_F_Mass}"/>
-			<box_inertia
-				m="${suspension_arm_F_Mass}"
-				x="${suspension_arm_F_Width*scale_XYZ}"
-				y="${suspension_arm_F_Length*scale_XYZ}"
-				z="${suspension_arm_F_Height*scale_XYZ}"/>
-		</inertial>
-	</link>
-  	<joint name="suspension_arm_B_R_joint" type="revolute">
-		<parent link="right_axis"/>
-		<child link="suspension_arm_B_R"/>
-		<origin xyz="0 0 0" rpy="0 0 0"/>
-		<limit lower="-0.2" upper="0.2" effort="10000.0" velocity="100.0"/>
-        <axis xyz="1 0 0"/>
-	</joint>
-  	<link name='suspension_arm_B_R_to_B2_R'>
-		<inertial>
-            <origin xyz="0 0 0" rpy="0 0 0"/>
-            <mass value="0.02" />
-            <inertia ixx="2.61666666667e-05" ixy="0.0" ixz="0.0" iyy="2.61666666667e-05" iyz="0.0" izz="3.6e-05"/>
-        </inertial>
-        <collision>
-            <origin xyz="0 0 0.015" rpy="0 0 0"/>
-            <geometry>
-                <cylinder radius="0.06" length="0.035"/>
-            </geometry>
-        </collision>
-		<visual>
-            <origin rpy="0.0 1.57 0" xyz="0 0 0"/>
-            <geometry>
-                <cylinder radius="0.04" length="0.1"/>
-            </geometry>
-        </visual>
-	</link>
-	<joint name="suspension_arm_B_R_to_B2_R_joint" type="fixed">
-		<parent link="suspension_arm_B_R"/>
-		<child link="suspension_arm_B_R_to_B2_R"/>
-		<origin xyz="0.05159 0.73683 -0.22972" rpy="0 -0.1937315 0"/>
-	</joint>
-	<link name='suspension_arm_B2_R'>
-		<collision>
-			<origin xyz="0 0 0"
-					rpy="0 0 0"/>
-			<geometry>
-				<mesh filename="package://curiosity_mars_rover_description/meshes/suspension_arm_B2_R_fixed.dae" scale="${scale_XYZ} ${scale_XYZ} ${scale_XYZ}"/>
-			</geometry>
-		</collision>
-		<visual>
-			<origin xyz="0 0 0"
-					rpy="0 0 0"/>
-			<geometry>
-				<mesh filename="package://curiosity_mars_rover_description/meshes/suspension_arm_B2_R_fixed.dae" scale="${scale_XYZ} ${scale_XYZ} ${scale_XYZ}"/>
-			</geometry>
-		</visual>
-		<inertial>
-			<origin xyz="0 0 0"
-					rpy="0 0 0"/>
-			<mass value="${suspension_arm_F_Mass}"/>
-			<box_inertia
-				m="${suspension_arm_F_Mass}"
-				x="${suspension_arm_F_Width*scale_XYZ}"
-				y="${suspension_arm_F_Length*scale_XYZ}"
-				z="${suspension_arm_F_Height*scale_XYZ}"/>
-		</inertial>
-	</link>
-  	<joint name="suspension_arm_B2_R_joint" type="revolute">
-		<parent link="suspension_arm_B_R_to_B2_R"/>
-		<child link="suspension_arm_B2_R"/>
-		<origin xyz="0 0 0" rpy="0 0 0"/>
-		<limit lower="-0.2" upper="0.2" effort="10000.0" velocity="100.0"/>
-        <axis xyz="1 0 0"/>
-	</joint>
   </xacro:macro>
 </robot>

File: curiosity_mars_rover_description/urdf/curiosity_mars_rover_properties.xacro (robot description, xacro)
@@ -6,28 +6,76 @@
 	<xacro:property name="scale_XYZ" value="1.0"/>
 	<!-- Chassis properties -->
-	<!--
-	<xacro:property name="chassisHeight" value="0.76"/>
-	<xacro:property name="chassisLength" value="1.53774"/>
-	<xacro:property name="chassisWidth" value="2.08157"/>
-	-->
+	<xacro:property name="chassisMass" value="733.64"/>
 	<xacro:property name="chassisHeight" value="0.76"/>
 	<xacro:property name="chassisLength" value="2.08157"/>
 	<xacro:property name="chassisWidth" value="1.53774"/>
-	<xacro:property name="chassisMass" value="20.0"/>
+	<!-- Wheel Trees -->
+	<xacro:property name="TreeMass" value="${72.96/2.0}"/>
+	<xacro:property name="TreeParts" value="5.0"/>
 	<xacro:property name="axisHeight" value="0.36388"/>
 	<xacro:property name="axisLength" value="0.20321"/>
 	<xacro:property name="axisWidth" value="0.27070"/>
-	<xacro:property name="axisMass" value="20.0"/>
-	<xacro:property name="suspension_arm_F_Height" value="0.30536"/>
-	<xacro:property name="suspension_arm_F_Length" value="1.02203"/>
-	<xacro:property name="suspension_arm_F_Width" value="0.39606"/>
-	<xacro:property name="suspension_arm_F_Mass" value="20.0"/>
-	<xacro:property name="armHeight" value="0.01"/>
-	<xacro:property name="armLength" value="0.01"/>
-	<xacro:property name="armWidth" value="0.01"/>
-	<xacro:property name="armMass" value="0.01"/>
-	<!-- Differential-drive wheels properties -->
+	<xacro:property name="axisMass" value="${TreeMass/TreeParts}"/>
+	<xacro:property name="suspension_arm_F_L_Mass" value="${TreeMass/TreeParts}"/>
+	<xacro:property name="suspension_arm_F_L_X" value="0.39606"/>
+	<xacro:property name="suspension_arm_F_L_Y" value="1.02203"/>
+	<xacro:property name="suspension_arm_F_L_Z" value="0.30536"/>
+	<xacro:property name="suspension_arm_B_L_Mass" value="${TreeMass/TreeParts}"/>
+	<xacro:property name="suspension_arm_B_L_X" value="0.123524"/>
+	<xacro:property name="suspension_arm_B_L_Y" value="0.852108"/>
+	<xacro:property name="suspension_arm_B_L_Z" value="0.348354"/>
+	<xacro:property name="suspension_arm_B2_L_Mass" value="${TreeMass/TreeParts}"/>
+	<xacro:property name="suspension_arm_B2_L_X" value="0.400262"/>
+	<xacro:property name="suspension_arm_B2_L_Y" value="1.22113"/>
+	<xacro:property name="suspension_arm_B2_L_Z" value="0.631338"/>
+	<xacro:property name="suspension_steer_F_L_Mass" value="${TreeMass/TreeParts}"/>
+	<xacro:property name="suspension_steer_F_L_X" value="0.528399"/>
+	<xacro:property name="suspension_steer_F_L_Y" value="0.21019"/>
+	<xacro:property name="suspension_steer_F_L_Z" value="0.450036"/>
+	<xacro:property name="suspension_steer_B_L_Mass" value="${TreeMass/TreeParts}"/>
+	<xacro:property name="suspension_steer_B_L_X" value="0.528399"/>
+	<xacro:property name="suspension_steer_B_L_Y" value="0.21019"/>
+	<xacro:property name="suspension_steer_B_L_Z" value="0.450036"/>
+	<!-- Wheels properties -->
 	<xacro:property name="wheelWidth" value="0.39473"/>
 	<xacro:property name="wheelRadius" value="0.242645"/>
-	<xacro:property name="wheelMass" value="0.05"/>
+	<xacro:property name="wheelMass" value="2.07"/>
+	<!-- Arm -->
+	<xacro:property name="armMass" value="30.0"/>
+	<xacro:property name="armParts" value="5.0"/>
+	<xacro:property name="arm_01_Mass" value="${armMass/armParts}"/>
+	<xacro:property name="arm_01_X" value="0.356891"/>
+	<xacro:property name="arm_01_Y" value="0.334128"/>
+	<xacro:property name="arm_01_Z" value="0.300511"/>
+	<xacro:property name="arm_02_Mass" value="${armMass/armParts}"/>
+	<xacro:property name="arm_02_X" value="0.472171"/>
+	<xacro:property name="arm_02_Y" value="0.972313"/>
+	<xacro:property name="arm_02_Z" value="0.218611"/>
+	<xacro:property name="arm_03_Mass" value="${armMass/armParts}"/>
+	<xacro:property name="arm_03_X" value="0.30683"/>
+	<xacro:property name="arm_03_Y" value="0.178607"/>
+	<xacro:property name="arm_03_Z" value="0.878958"/>
+	<xacro:property name="arm_04_Mass" value="${armMass/armParts}"/>
+	<xacro:property name="arm_04_X" value="0.32452"/>
+	<xacro:property name="arm_04_Y" value="0.344693"/>
+	<xacro:property name="arm_04_Z" value="0.288832"/>
+	<xacro:property name="arm_tools_Mass" value="${armMass/armParts}"/>
+	<xacro:property name="arm_tools_X" value="0.60282"/>
+	<xacro:property name="arm_tools_Y" value="0.467147"/>
+	<xacro:property name="arm_tools_Z" value="0.21915"/>
+	<!-- Mast -->
+	<xacro:property name="mastMass" value="50.0"/>
+	<xacro:property name="MastParts" value="3.0"/>
+	<xacro:property name="mast_p_Mass" value="${mastMass/MastParts}"/>
+	<xacro:property name="mast_p_X" value="0.192274"/>
+	<xacro:property name="mast_p_Y" value="0.221494"/>
+	<xacro:property name="mast_p_Z" value="0.525621"/>
+	<xacro:property name="mast_02_Mass" value="${mastMass/MastParts}"/>
+	<xacro:property name="mast_02_X" value="0.270963"/>
+	<xacro:property name="mast_02_Y" value="0.232093"/>
+	<xacro:property name="mast_02_Z" value="0.285976"/>
+	<xacro:property name="mast_cameras_Mass" value="${mastMass/MastParts}"/>
+	<xacro:property name="mast_cameras_X" value="0.550001"/>
+	<xacro:property name="mast_cameras_Y" value="0.283001"/>
+	<xacro:property name="mast_cameras_Z" value="0.203994"/>
 </robot>
