Commit message: Added correct innertias and masses

File: curiosity_mars_rover_description/urdf/left_wheel_group.xacro (robot description, xacro)
@@ -2,4 +2,158 @@
 <robot xmlns:xacro="http://www.ros.org/wiki/xacro">
   <xacro:macro name="left_wheel_tree" params="">
+  	<link name='left_axis'>
+		<collision>
+			<origin xyz="0 0 0"
+					rpy="0 0 0"/>
+			<geometry>
+				<mesh filename="package://curiosity_mars_rover_description/meshes/left_axis_jointfix_v2.dae" scale="${scale_XYZ} ${scale_XYZ} ${scale_XYZ}"/>
+			</geometry>
+		</collision>
+		<visual>
+			<origin xyz="0 0 0"
+					rpy="0 0 0"/>
+			<geometry>
+				<mesh filename="package://curiosity_mars_rover_description/meshes/left_axis_jointfix_v2.dae" scale="${scale_XYZ} ${scale_XYZ} ${scale_XYZ}"/>
+			</geometry>
+		</visual>
+		<inertial>
+			<origin xyz="0 0 0"
+					rpy="0 0 0"/>
+			<mass value="${axisMass}"/>
+			<box_inertia
+				m="${axisMass}"
+				x="${axisWidth*scale_XYZ}"
+				y="${axisLength*scale_XYZ}"
+				z="${axisHeight*scale_XYZ}"/>
+		</inertial>
+	</link>
+  	<joint name="left_axis_joint" type="fixed">
+		<parent link="chassis"/>
+		<child link="left_axis"/>
+		<origin xyz="0.7938 -0.2133 0" rpy="0 -0.19565141 0"/>
+	</joint>
+  	<link name='suspension_arm_F_L'>
+		<collision>
+			<origin xyz="0 0 0"
+					rpy="0 0 0"/>
+			<geometry>
+				<mesh filename="package://curiosity_mars_rover_description/meshes/suspension_arm_F_L_fixed.dae" scale="${scale_XYZ} ${scale_XYZ} ${scale_XYZ}"/>
+			</geometry>
+		</collision>
+		<visual>
+			<origin xyz="0 0 0"
+					rpy="0 0 0"/>
+			<geometry>
+				<mesh filename="package://curiosity_mars_rover_description/meshes/suspension_arm_F_L_fixed.dae" scale="${scale_XYZ} ${scale_XYZ} ${scale_XYZ}"/>
+			</geometry>
+		</visual>
+		<inertial>
+			<origin xyz="0 0 0"
+					rpy="0 0 0"/>
+			<mass value="${suspension_arm_F_L_Mass}"/>
+			<box_inertia
+				m="${suspension_arm_F_L_Mass}"
+				x="${suspension_arm_F_L_X*scale_XYZ}"
+				y="${suspension_arm_F_L_Y*scale_XYZ}"
+				z="${suspension_arm_F_L_Z*scale_XYZ}"/>
+		</inertial>
+	</link>
+  	<joint name="suspension_arm_F_L_joint" type="revolute">
+		<parent link="left_axis"/>
+		<child link="suspension_arm_F_L"/>
+		<origin xyz="0 0 0" rpy="0 0 0"/>
+		<limit lower="-0.2" upper="0.2" effort="10000.0" velocity="100.0"/>
+        <axis xyz="1 0 0"/>
+	</joint>
+  	<link name='suspension_arm_B_L'>
+		<collision>
+			<origin xyz="0 0 0"
+					rpy="0 0 0"/>
+			<geometry>
+				<mesh filename="package://curiosity_mars_rover_description/meshes/suspension_arm_B_L_fixed.dae" scale="${scale_XYZ} ${scale_XYZ} ${scale_XYZ}"/>
+			</geometry>
+		</collision>
+		<visual>
+			<origin xyz="0 0 0"
+					rpy="0 0 0"/>
+			<geometry>
+				<mesh filename="package://curiosity_mars_rover_description/meshes/suspension_arm_B_L_fixed.dae" scale="${scale_XYZ} ${scale_XYZ} ${scale_XYZ}"/>
+			</geometry>
+		</visual>
+		<inertial>
+			<origin xyz="0 0 0"
+					rpy="0 0 0"/>
+			<mass value="${suspension_arm_B_L_Mass}"/>
+			<box_inertia
+				m="${suspension_arm_B_L_Mass}"
+				x="${suspension_arm_B_L_X*scale_XYZ}"
+				y="${suspension_arm_B_L_Y*scale_XYZ}"
+				z="${suspension_arm_B_L_Z*scale_XYZ}"/>
+		</inertial>
+	</link>
+  	<joint name="suspension_arm_B_L_joint" type="revolute">
+		<parent link="left_axis"/>
+		<child link="suspension_arm_B_L"/>
+		<origin xyz="0 0 0" rpy="0 0 0"/>
+		<limit lower="-0.2" upper="0.2" effort="10000.0" velocity="100.0"/>
+        <axis xyz="1 0 0"/>
+	</joint>
+ 	<link name='suspension_arm_B_L_to_B2_L'>
+		<inertial>
+            <origin xyz="0 0 0" rpy="0 0 0"/>
+            <mass value="0.02" />
+            <inertia ixx="2.61666666667e-05" ixy="0.0" ixz="0.0" iyy="2.61666666667e-05" iyz="0.0" izz="3.6e-05"/>
+        </inertial>
+        <collision>
+            <origin xyz="0 0 0.015" rpy="0 0 0"/>
+            <geometry>
+                <cylinder radius="0.06" length="0.035"/>
+            </geometry>
+        </collision>
+		<visual>
+            <origin rpy="0.0 1.57 0" xyz="0 0 0"/>
+            <geometry>
+                <cylinder radius="0.04" length="0.1"/>
+            </geometry>
+        </visual>
+	</link>
+	<joint name="suspension_arm_B_L_to_B2_L_joint" type="fixed">
+		<parent link="suspension_arm_B_L"/>
+		<child link="suspension_arm_B_L_to_B2_L"/>
+		<origin xyz="-0.05159 0.73683 -0.22972" rpy="0 0.1937315 0"/>
+	</joint>
+	<link name='suspension_arm_B2_L'>
+		<collision>
+			<origin xyz="0 0 0"
+					rpy="0 0 0"/>
+			<geometry>
+				<mesh filename="package://curiosity_mars_rover_description/meshes/suspension_arm_B2_L_fixed.dae" scale="${scale_XYZ} ${scale_XYZ} ${scale_XYZ}"/>
+			</geometry>
+		</collision>
+		<visual>
+			<origin xyz="0 0 0"
+					rpy="0 0 0"/>
+			<geometry>
+				<mesh filename="package://curiosity_mars_rover_description/meshes/suspension_arm_B2_L_fixed.dae" scale="${scale_XYZ} ${scale_XYZ} ${scale_XYZ}"/>
+			</geometry>
+		</visual>
+		<inertial>
+			<origin xyz="0 0 0"
+					rpy="0 0 0"/>
+			<mass value="${suspension_arm_B2_L_Mass}"/>
+			<box_inertia
+				m="${suspension_arm_B2_L_Mass}"
+				x="${suspension_arm_B2_L_X*scale_XYZ}"
+				y="${suspension_arm_B2_L_Y*scale_XYZ}"
+				z="${suspension_arm_B2_L_Z*scale_XYZ}"/>
+		</inertial>
+	</link>
+  	<joint name="suspension_arm_B2_L_joint" type="revolute">
+		<parent link="suspension_arm_B_L_to_B2_L"/>
+		<child link="suspension_arm_B2_L"/>
+		<origin xyz="0 0 0" rpy="0 0 0"/>
+		<limit lower="-0.2" upper="0.2" effort="10000.0" velocity="100.0"/>
+        <axis xyz="1 0 0"/>
+	</joint>
 	<!-- FRONT WHEEL -->
 	<link name='suspension_arm_F_L_to_suspension_steer_F_L'>
@@ -45,10 +199,10 @@
 			<origin xyz="0 0 0"
 					rpy="0 0 0"/>
-			<mass value="${suspension_arm_F_Mass}"/>
-			<box_inertia
-				m="${suspension_arm_F_Mass}"
-				x="${suspension_arm_F_Width*scale_XYZ}"
-				y="${suspension_arm_F_Length*scale_XYZ}"
-				z="${suspension_arm_F_Height*scale_XYZ}"/>
+			<mass value="${suspension_steer_F_L_Mass}"/>
+			<box_inertia
+				m="${suspension_steer_F_L_Mass}"
+				x="${suspension_steer_F_L_X*scale_XYZ}"
+				y="${suspension_steer_F_L_Y*scale_XYZ}"
+				z="${suspension_steer_F_L_Z*scale_XYZ}"/>
 		</inertial>
 	</link>
@@ -162,10 +316,10 @@
 			<origin xyz="0 0 0"
 					rpy="0 0 0"/>
-			<mass value="${suspension_arm_F_Mass}"/>
-			<box_inertia
-				m="${suspension_arm_F_Mass}"
-				x="${suspension_arm_F_Width*scale_XYZ}"
-				y="${suspension_arm_F_Length*scale_XYZ}"
-				z="${suspension_arm_F_Height*scale_XYZ}"/>
+			<mass value="${suspension_steer_B_L_Mass}"/>
+			<box_inertia
+				m="${suspension_steer_B_L_Mass}"
+				x="${suspension_steer_B_L_X*scale_XYZ}"
+				y="${suspension_steer_B_L_Y*scale_XYZ}"
+				z="${suspension_steer_B_L_Z*scale_XYZ}"/>
 		</inertial>
 	</link>

File: curiosity_mars_rover_description/urdf/right_wheel_group.xacro (robot description, xacro)
@@ -2,4 +2,158 @@
 <robot xmlns:xacro="http://www.ros.org/wiki/xacro">
   <xacro:macro name="right_wheel_tree" params="">
+  	<link name='right_axis'>
+		<collision>
+			<origin xyz="0 0 0"
+					rpy="0 0 0"/>
+			<geometry>
+				<mesh filename="package://curiosity_mars_rover_description/meshes/right_axis_jointfix_v2.dae" scale="${scale_XYZ} ${scale_XYZ} ${scale_XYZ}"/>
+			</geometry>
+		</collision>
+		<visual>
+			<origin xyz="0 0 0"
+					rpy="0 0 0"/>
+			<geometry>
+				<mesh filename="package://curiosity_mars_rover_description/meshes/right_axis_jointfix_v2.dae" scale="${scale_XYZ} ${scale_XYZ} ${scale_XYZ}"/>
+			</geometry>
+		</visual>
+		<inertial>
+			<origin xyz="0 0 0"
+					rpy="0 0 0"/>
+			<mass value="${axisMass}"/>
+			<box_inertia
+				m="${axisMass}"
+				x="${axisWidth*scale_XYZ}"
+				y="${axisLength*scale_XYZ}"
+				z="${axisHeight*scale_XYZ}"/>
+		</inertial>
+	</link>
+  	<joint name="right_axis_joint" type="fixed">
+		<parent link="chassis"/>
+		<child link="right_axis"/>
+		<origin xyz="-0.7938 -0.2133 0" rpy="0 0.19565141 0"/>
+	</joint>
+	<link name='suspension_arm_F_R'>
+		<collision>
+			<origin xyz="0 0 0"
+					rpy="0 0 0"/>
+			<geometry>
+				<mesh filename="package://curiosity_mars_rover_description/meshes/suspension_arm_F_R_fixed.dae" scale="${scale_XYZ} ${scale_XYZ} ${scale_XYZ}"/>
+			</geometry>
+		</collision>
+		<visual>
+			<origin xyz="0 0 0"
+					rpy="0 0 0"/>
+			<geometry>
+				<mesh filename="package://curiosity_mars_rover_description/meshes/suspension_arm_F_R_fixed.dae" scale="${scale_XYZ} ${scale_XYZ} ${scale_XYZ}"/>
+			</geometry>
+		</visual>
+		<inertial>
+			<origin xyz="0 0 0"
+					rpy="0 0 0"/>
+			<mass value="${suspension_arm_F_L_Mass}"/>
+			<box_inertia
+				m="${suspension_arm_F_L_Mass}"
+				x="${suspension_arm_F_L_X*scale_XYZ}"
+				y="${suspension_arm_F_L_Y*scale_XYZ}"
+				z="${suspension_arm_F_L_Z*scale_XYZ}"/>
+		</inertial>
+	</link>
+  	<joint name="suspension_arm_F_R_joint" type="revolute">
+		<parent link="right_axis"/>
+		<child link="suspension_arm_F_R"/>
+		<origin xyz="0 0 0" rpy="0 0 0"/>
+		<limit lower="-0.2" upper="0.2" effort="10000.0" velocity="100.0"/>
+        <axis xyz="1 0 0"/>
+	</joint>
+  	<link name='suspension_arm_B_R'>
+		<collision>
+			<origin xyz="0 0 0"
+					rpy="0 0 0"/>
+			<geometry>
+				<mesh filename="package://curiosity_mars_rover_description/meshes/suspension_arm_B_R_fixed.dae" scale="${scale_XYZ} ${scale_XYZ} ${scale_XYZ}"/>
+			</geometry>
+		</collision>
+		<visual>
+			<origin xyz="0 0 0"
+					rpy="0 0 0"/>
+			<geometry>
+				<mesh filename="package://curiosity_mars_rover_description/meshes/suspension_arm_B_R_fixed.dae" scale="${scale_XYZ} ${scale_XYZ} ${scale_XYZ}"/>
+			</geometry>
+		</visual>
+		<inertial>
+			<origin xyz="0 0 0"
+					rpy="0 0 0"/>
+			<mass value="${suspension_arm_B_L_Mass}"/>
+			<box_inertia
+				m="${suspension_arm_B_L_Mass}"
+				x="${suspension_arm_B_L_X*scale_XYZ}"
+				y="${suspension_arm_B_L_Y*scale_XYZ}"
+				z="${suspension_arm_B_L_Z*scale_XYZ}"/>
+		</inertial>
+	</link>
+  	<joint name="suspension_arm_B_R_joint" type="revolute">
+		<parent link="right_axis"/>
+		<child link="suspension_arm_B_R"/>
+		<origin xyz="0 0 0" rpy="0 0 0"/>
+		<limit lower="-0.2" upper="0.2" effort="10000.0" velocity="100.0"/>
+        <axis xyz="1 0 0"/>
+	</joint>
+  	<link name='suspension_arm_B_R_to_B2_R'>
+		<inertial>
+            <origin xyz="0 0 0" rpy="0 0 0"/>
+            <mass value="0.02" />
+            <inertia ixx="2.61666666667e-05" ixy="0.0" ixz="0.0" iyy="2.61666666667e-05" iyz="0.0" izz="3.6e-05"/>
+        </inertial>
+        <collision>
+            <origin xyz="0 0 0.015" rpy="0 0 0"/>
+            <geometry>
+                <cylinder radius="0.06" length="0.035"/>
+            </geometry>
+        </collision>
+		<visual>
+            <origin rpy="0.0 1.57 0" xyz="0 0 0"/>
+            <geometry>
+                <cylinder radius="0.04" length="0.1"/>
+            </geometry>
+        </visual>
+	</link>
+	<joint name="suspension_arm_B_R_to_B2_R_joint" type="fixed">
+		<parent link="suspension_arm_B_R"/>
+		<child link="suspension_arm_B_R_to_B2_R"/>
+		<origin xyz="0.05159 0.73683 -0.22972" rpy="0 -0.1937315 0"/>
+	</joint>
+	<link name='suspension_arm_B2_R'>
+		<collision>
+			<origin xyz="0 0 0"
+					rpy="0 0 0"/>
+			<geometry>
+				<mesh filename="package://curiosity_mars_rover_description/meshes/suspension_arm_B2_R_fixed.dae" scale="${scale_XYZ} ${scale_XYZ} ${scale_XYZ}"/>
+			</geometry>
+		</collision>
+		<visual>
+			<origin xyz="0 0 0"
+					rpy="0 0 0"/>
+			<geometry>
+				<mesh filename="package://curiosity_mars_rover_description/meshes/suspension_arm_B2_R_fixed.dae" scale="${scale_XYZ} ${scale_XYZ} ${scale_XYZ}"/>
+			</geometry>
+		</visual>
+		<inertial>
+			<origin xyz="0 0 0"
+					rpy="0 0 0"/>
+			<mass value="${suspension_arm_B2_L_Mass}"/>
+			<box_inertia
+				m="${suspension_arm_B2_L_Mass}"
+				x="${suspension_arm_B2_L_X*scale_XYZ}"
+				y="${suspension_arm_B2_L_Y*scale_XYZ}"
+				z="${suspension_arm_B2_L_Z*scale_XYZ}"/>
+		</inertial>
+	</link>
+  	<joint name="suspension_arm_B2_R_joint" type="revolute">
+		<parent link="suspension_arm_B_R_to_B2_R"/>
+		<child link="suspension_arm_B2_R"/>
+		<origin xyz="0 0 0" rpy="0 0 0"/>
+		<limit lower="-0.2" upper="0.2" effort="10000.0" velocity="100.0"/>
+        <axis xyz="1 0 0"/>
+	</joint>
 	<!-- FRONT WHEEL RIGHT -->
 	<link name='suspension_arm_F_R_to_suspension_steer_F_R'>
@@ -45,10 +199,10 @@
 			<origin xyz="0 0 0"
 					rpy="0 0 0"/>
-			<mass value="${suspension_arm_F_Mass}"/>
-			<box_inertia
-				m="${suspension_arm_F_Mass}"
-				x="${suspension_arm_F_Width*scale_XYZ}"
-				y="${suspension_arm_F_Length*scale_XYZ}"
-				z="${suspension_arm_F_Height*scale_XYZ}"/>
+			<mass value="${suspension_steer_F_L_Mass}"/>
+			<box_inertia
+				m="${suspension_steer_F_L_Mass}"
+				x="${suspension_steer_F_L_X*scale_XYZ}"
+				y="${suspension_steer_F_L_Y*scale_XYZ}"
+				z="${suspension_steer_F_L_Z*scale_XYZ}"/>
 		</inertial>
 	</link>
@@ -160,10 +314,10 @@
 			<origin xyz="0 0 0"
 					rpy="0 0 0"/>
-			<mass value="${suspension_arm_F_Mass}"/>
-			<box_inertia
-				m="${suspension_arm_F_Mass}"
-				x="${suspension_arm_F_Width*scale_XYZ}"
-				y="${suspension_arm_F_Length*scale_XYZ}"
-				z="${suspension_arm_F_Height*scale_XYZ}"/>
+			<mass value="${suspension_steer_B_L_Mass}"/>
+			<box_inertia
+				m="${suspension_steer_B_L_Mass}"
+				x="${suspension_steer_B_L_X*scale_XYZ}"
+				y="${suspension_steer_B_L_Y*scale_XYZ}"
+				z="${suspension_steer_B_L_Z*scale_XYZ}"/>
 		</inertial>
 	</link>

File: curiosity_mars_rover_description/urdf/sensor_mast.xacro (robot description, xacro)
@@ -44,10 +44,10 @@
 			<origin xyz="0 0 0"
 					rpy="0 0 0"/>
-			<mass value="${armMass}"/>
+			<mass value="${mast_p_Mass}"/>
 			<box_inertia
-				m="${armMass}"
-				x="${armWidth*scale_XYZ}"
-				y="${armLength*scale_XYZ}"
-				z="${armHeight*scale_XYZ}"/>
+				m="${mast_p_Mass}"
+				x="${mast_p_X*scale_XYZ}"
+				y="${mast_p_Y*scale_XYZ}"
+				z="${mast_p_Z*scale_XYZ}"/>
 		</inertial>
 	</link>
@@ -57,5 +57,5 @@
 		<origin xyz="0 0 0" rpy="0 0 0"/>
 		<limit lower="-0.2" upper="0.2" effort="10000.0" velocity="100.0"/>
-        <axis xyz="0 0 1"/>
+        <axis xyz="0 1 0"/>
         <joint_properties damping="0.0" friction="0.0"/>
 	</joint>
@@ -66,4 +66,140 @@
       </joint>
       <actuator name="mast_pMotor">
+        <hardwareInterface>hardware_interface/EffortJointInterface</hardwareInterface>
+        <mechanicalReduction>1</mechanicalReduction>
+      </actuator>
+    </transmission>
+  	<link name='mast_p_to_mast_02'>
+		<inertial>
+            <origin xyz="0 0 0" rpy="0 0 0"/>
+            <mass value="0.02" />
+            <inertia ixx="2.61666666667e-05" ixy="0.0" ixz="0.0" iyy="2.61666666667e-05" iyz="0.0" izz="3.6e-05"/>
+        </inertial>
+        <collision>
+            <origin rpy="0 0 0" xyz="0 0 0"/>
+            <geometry>
+                <cylinder radius="0.02" length="0.02"/>
+            </geometry>
+        </collision>
+		<visual>
+            <origin rpy="0 0 0" xyz="0 0 0"/>
+            <geometry>
+                <cylinder radius="0.02" length="0.02"/>
+            </geometry>
+        </visual>
+	</link>
+	<joint name="mast_p_to_mast_02_joint" type="fixed">
+		<parent link="mast_p"/>
+		<child link="mast_p_to_mast_02"/>
+		<origin xyz="0 0 0.473641" rpy="0 0 0"/>
+	</joint>
+	<link name='mast_02'>
+		<collision>
+			<origin xyz="0 0 0"
+					rpy="0 0 0"/>
+			<geometry>
+				<mesh filename="package://curiosity_mars_rover_description/meshes/mast_02_fixed.dae" scale="${scale_XYZ} ${scale_XYZ} ${scale_XYZ}"/>
+			</geometry>
+		</collision>
+		<visual>
+			<origin xyz="0 0 0"
+					rpy="0 0 0"/>
+			<geometry>
+				<mesh filename="package://curiosity_mars_rover_description/meshes/mast_02_fixed.dae" scale="${scale_XYZ} ${scale_XYZ} ${scale_XYZ}"/>
+			</geometry>
+		</visual>
+		<inertial>
+			<origin xyz="0 0 0"
+					rpy="0 0 0"/>
+			<mass value="${mast_02_Mass}"/>
+			<box_inertia
+				m="${mast_02_Mass}"
+				x="${mast_02_X*scale_XYZ}"
+				y="${mast_02_Y*scale_XYZ}"
+				z="${mast_02_Z*scale_XYZ}"/>
+		</inertial>
+	</link>
+  	<joint name="mast_02_joint" type="revolute">
+		<parent link="mast_p_to_mast_02"/>
+		<child link="mast_02"/>
+		<origin xyz="0 0 0" rpy="0 0 0"/>
+		<limit lower="-0.2" upper="0.2" effort="10000.0" velocity="100.0"/>
+        <axis xyz="0 0 1"/>
+        <joint_properties damping="0.0" friction="0.0"/>
+	</joint>
+    <transmission name="mast_02_trans">
+      <type>transmission_interface/SimpleTransmission</type>
+      <joint name="mast_02_joint">
+        <hardwareInterface>hardware_interface/EffortJointInterface</hardwareInterface>
+      </joint>
+      <actuator name="mast_02Motor">
+        <hardwareInterface>hardware_interface/EffortJointInterface</hardwareInterface>
+        <mechanicalReduction>1</mechanicalReduction>
+      </actuator>
+    </transmission>
+	<link name='mast_02_to_mast_cameras'>
+		<inertial>
+            <origin xyz="0 0 0" rpy="0 0 0"/>
+            <mass value="0.02" />
+            <inertia ixx="2.61666666667e-05" ixy="0.0" ixz="0.0" iyy="2.61666666667e-05" iyz="0.0" izz="3.6e-05"/>
+        </inertial>
+        <collision>
+            <origin rpy="0 0 0" xyz="0 0 0"/>
+            <geometry>
+                <cylinder radius="0.02" length="0.02"/>
+            </geometry>
+        </collision>
+		<visual>
+            <origin rpy="0 0 0" xyz="0 0 0"/>
+            <geometry>
+                <cylinder radius="0.02" length="0.02"/>
+            </geometry>
+        </visual>
+	</link>
+	<joint name="mast_02_to_mast_cameras_joint" type="fixed">
+		<parent link="mast_02"/>
+		<child link="mast_02_to_mast_cameras"/>
+		<origin xyz="0 0 0.20859" rpy="0 0 0"/>
+	</joint>
+	<link name='mast_cameras'>
+		<collision>
+			<origin xyz="0 0 0"
+					rpy="0 0 0"/>
+			<geometry>
+				<mesh filename="package://curiosity_mars_rover_description/meshes/mast_cameras.dae" scale="${scale_XYZ} ${scale_XYZ} ${scale_XYZ}"/>
+			</geometry>
+		</collision>
+		<visual>
+			<origin xyz="0 0 0"
+					rpy="0 0 0"/>
+			<geometry>
+				<mesh filename="package://curiosity_mars_rover_description/meshes/mast_cameras.dae" scale="${scale_XYZ} ${scale_XYZ} ${scale_XYZ}"/>
+			</geometry>
+		</visual>
+		<inertial>
+			<origin xyz="0 0 0"
+					rpy="0 0 0"/>
+			<mass value="${mast_cameras_Mass}"/>
+			<box_inertia
+				m="${mast_cameras_Mass}"
+				x="${mast_cameras_X*scale_XYZ}"
+				y="${mast_cameras_Y*scale_XYZ}"
+				z="${mast_cameras_Z*scale_XYZ}"/>
+		</inertial>
+	</link>
+  	<joint name="mast_cameras_joint" type="revolute">
+		<parent link="mast_02_to_mast_cameras"/>
+		<child link="mast_cameras"/>
+		<origin xyz="0 0 0" rpy="0 0 0"/>
+		<limit lower="-0.2" upper="0.2" effort="10000.0" velocity="100.0"/>
+        <axis xyz="1 0 0"/>
+        <joint_properties damping="0.0" friction="0.0"/>
+	</joint>
+    <transmission name="mast_02_trans">
+      <type>transmission_interface/SimpleTransmission</type>
+      <joint name="mast_cameras_joint">
+        <hardwareInterface>hardware_interface/EffortJointInterface</hardwareInterface>
+      </joint>
+      <actuator name="mast_02Motor">
         <hardwareInterface>hardware_interface/EffortJointInterface</hardwareInterface>
         <mechanicalReduction>1</mechanicalReduction>
