Commit message: Added stable version with cameras and services and rviz launch

File: curiosity_mars_rover_description/urdf/arm.xacro (robot description, xacro)
@@ -56,5 +56,5 @@
 		<child link="arm_01"/>
 		<origin xyz="0 0 0" rpy="0 0 0"/>
-		<limit lower="-0.2" upper="0.2" effort="10000.0" velocity="100.0"/>
+		<limit lower="${-arm_01_limit}" upper="${arm_01_limit}" effort="10000.0" velocity="100.0"/>
         <axis xyz="0 0 1"/>
         <joint_properties damping="0.0" friction="0.0"/>
@@ -124,5 +124,5 @@
 		<child link="arm_02"/>
 		<origin xyz="0 0 0" rpy="0 0 0"/>
-		<limit lower="-0.2" upper="0.2" effort="10000.0" velocity="100.0"/>
+		<limit lower="${-arm_02_limit}" upper="${arm_02_limit}" effort="10000.0" velocity="100.0"/>
         <axis xyz="1 0 0"/>
         <joint_properties damping="0.0" friction="0.0"/>
@@ -192,5 +192,5 @@
 		<child link="arm_03"/>
 		<origin xyz="0 0 0" rpy="0 0 0"/>
-		<limit lower="-0.2" upper="0.2" effort="10000.0" velocity="100.0"/>
+		<limit lower="${-arm_03_limit}" upper="${arm_03_limit}" effort="10000.0" velocity="100.0"/>
         <axis xyz="1 0 0"/>
         <joint_properties damping="0.0" friction="0.0"/>
@@ -260,5 +260,5 @@
 		<child link="arm_04"/>
 		<origin xyz="0 0 0" rpy="0 0 0"/>
-		<limit lower="-0.2" upper="0.2" effort="10000.0" velocity="100.0"/>
+		<limit lower="${-arm_04_limit}" upper="${arm_04_limit}" effort="10000.0" velocity="100.0"/>
         <axis xyz="0 1 0"/>
         <joint_properties damping="0.0" friction="0.0"/>
@@ -324,9 +324,9 @@
 		</inertial>
 	</link>
-  	<joint name="arm_tools_joint" type="revolute">
+  	<joint name="arm_tools_joint" type="continuous">
 		<parent link="arm_04_to_arm_tools"/>
 		<child link="arm_tools"/>
 		<origin xyz="0 0 0" rpy="0 0 0"/>
-		<limit lower="-0.2" upper="0.2" effort="10000.0" velocity="100.0"/>
+		<limit effort="10000.0" velocity="100.0"/>
         <axis xyz="0 0 1"/>
         <joint_properties damping="0.0" friction="0.0"/>

File: curiosity_mars_rover_description/urdf/curiosity_mars_rover.xacro (robot description, xacro)
@@ -20,7 +20,5 @@
 	<left_wheel_tree/>
 	<right_wheel_tree/>
-	<!--
 	<arm/>
 	<sensor_mast/>
-	-->
 </robot>

File: curiosity_mars_rover_description/urdf/curiosity_mars_rover_properties.xacro (robot description, xacro)
@@ -59,16 +59,20 @@
 	<xacro:property name="arm_01_Y" value="0.334128"/>
 	<xacro:property name="arm_01_Z" value="0.300511"/>
+	<xacro:property name="arm_01_limit" value="1.57"/>
 	<xacro:property name="arm_02_Mass" value="${armMass/armParts}"/>
 	<xacro:property name="arm_02_X" value="0.472171"/>
 	<xacro:property name="arm_02_Y" value="0.972313"/>
 	<xacro:property name="arm_02_Z" value="0.218611"/>
+	<xacro:property name="arm_02_limit" value="1.57"/>
 	<xacro:property name="arm_03_Mass" value="${armMass/armParts}"/>
 	<xacro:property name="arm_03_X" value="0.30683"/>
 	<xacro:property name="arm_03_Y" value="0.178607"/>
 	<xacro:property name="arm_03_Z" value="0.878958"/>
+	<xacro:property name="arm_03_limit" value="1.57"/>
 	<xacro:property name="arm_04_Mass" value="${armMass/armParts}"/>
 	<xacro:property name="arm_04_X" value="0.32452"/>
 	<xacro:property name="arm_04_Y" value="0.344693"/>
 	<xacro:property name="arm_04_Z" value="0.288832"/>
+	<xacro:property name="arm_04_limit" value="1.57"/>
 	<xacro:property name="arm_tools_Mass" value="${armMass/armParts}"/>
 	<xacro:property name="arm_tools_X" value="0.60282"/>
@@ -82,4 +86,6 @@
 	<xacro:property name="mast_p_Y" value="0.221494"/>
 	<xacro:property name="mast_p_Z" value="0.525621"/>
+	<xacro:property name="mast_p_upper_limit" value="1.57"/>
+	<xacro:property name="mast_p_lower_limit" value="0.0"/>
 	<xacro:property name="mast_02_Mass" value="${mastMass/MastParts}"/>
 	<xacro:property name="mast_02_X" value="0.270963"/>
@@ -90,3 +96,4 @@
 	<xacro:property name="mast_cameras_Y" value="0.283001"/>
 	<xacro:property name="mast_cameras_Z" value="0.203994"/>
+	<xacro:property name="mast_cameras_limit" value="1.57"/>
 </robot>

File: curiosity_mars_rover_description/urdf/sensor_mast.xacro (robot description, xacro)
@@ -56,5 +56,5 @@
 		<child link="mast_p"/>
 		<origin xyz="0 0 0" rpy="0 0 0"/>
-		<limit lower="-0.2" upper="0.2" effort="10000.0" velocity="100.0"/>
+		<limit lower="${mast_p_lower_limit}" upper="${mast_p_upper_limit}" effort="10000.0" velocity="100.0"/>
         <axis xyz="0 1 0"/>
         <joint_properties damping="0.0" friction="0.0"/>
@@ -120,9 +120,9 @@
 		</inertial>
 	</link>
-  	<joint name="mast_02_joint" type="revolute">
+  	<joint name="mast_02_joint" type="continuous">
 		<parent link="mast_p_to_mast_02"/>
 		<child link="mast_02"/>
 		<origin xyz="0 0 0" rpy="0 0 0"/>
-		<limit lower="-0.2" upper="0.2" effort="10000.0" velocity="100.0"/>
+		<limit effort="10000.0" velocity="100.0"/>
         <axis xyz="0 0 1"/>
         <joint_properties damping="0.0" friction="0.0"/>
@@ -192,5 +192,5 @@
 		<child link="mast_cameras"/>
 		<origin xyz="0 0 0" rpy="0 0 0"/>
-		<limit lower="-0.2" upper="0.2" effort="10000.0" velocity="100.0"/>
+		<limit lower="${-mast_cameras_limit}" upper="${mast_cameras_limit}" effort="10000.0" velocity="100.0"/>
         <axis xyz="1 0 0"/>
         <joint_properties damping="0.0" friction="0.0"/>
@@ -206,4 +206,30 @@
       </actuator>
     </transmission>
+  	<material name="green">
+        <color rgba="0 0.8 0 1"/>
+    </material>
+  	<link name="camera_link">
+        <!-- Inertial for gazebo to take it into account, Put 1gr weight -->
+        <inertial>
+            <origin xyz="0 0 0" rpy="0 0 0"/>
+            <mass value="0.001" />
+            <inertia ixx="9.1875e-09" ixy="0.0" ixz="0.0" iyy="9.1875e-09" iyz="0.0" izz="1.378125e-08"/>
+        </inertial>
+		<visual>
+            <origin rpy="0.0 0 0" xyz="0 0 0"/>
+            <geometry>
+                <box size="0.0005 0.0005 0.0005"/>
+            </geometry>
+            <material name="green"/>
+        </visual>
+	</link>
+    <gazebo reference="camera_link">
+        <material>Gazebo/Green</material>
+    </gazebo>
+    <joint name="head_camera_joint" type="fixed">
+        <parent link="mast_cameras"/>
+        <child link="camera_link"/>
+        <origin xyz="0.13642 -0.218683 0.222314" rpy="0 0 ${PI}"/>
+    </joint>
   </xacro:macro>
 </robot>
